Commit message: Updated urdf files and STL meshes. Includes scripts from Greg Lee.

File: abby_urdf/abby.urdf (robot description, URDF)
Before this commit: robot robot, 47 links, 46 joints
Links:
- removed link base_link
- removed link invacare assy:11
- added link battery rails:11, mass 0.429243531578; collision mesh filename=package://abby_urdf/battery rails_ipt_62ca575f.STL scale=0.0254 0.0254 0.0254; visual mesh filename=package://abby_urdf/battery rails_ipt_62ca575f.STL scale=0.0254 0.0254 0.0254
- added link battery:11, mass 21.545637575; collision mesh filename=package://abby_urdf/battery_ipt_8c19ab2.STL scale=0.0254 0.0254 0.0254; visual mesh filename=package://abby_urdf/battery_ipt_8c19ab2.STL scale=0.0254 0.0254 0.0254
- added link battery:21, mass 21.545637575; collision mesh filename=package://abby_urdf/battery_ipt_8c19ab2.STL scale=0.0254 0.0254 0.0254; visual mesh filename=package://abby_urdf/battery_ipt_8c19ab2.STL scale=0.0254 0.0254 0.0254
- added link caster wheel:11, mass 1.4177347039; collision mesh filename=package://abby_urdf/caster wheel_ipt_4784d7d8.STL scale=0.0254 0.0254 0.0254; visual mesh filename=package://abby_urdf/caster wheel_ipt_4784d7d8.STL scale=0.0254 0.0254 0.0254
- added link caster wheel:12, mass 1.4177347039; collision mesh filename=package://abby_urdf/caster wheel_ipt_4784d7d8.STL scale=0.0254 0.0254 0.0254; visual mesh filename=package://abby_urdf/caster wheel_ipt_4784d7d8.STL scale=0.0254 0.0254 0.0254
- added link caster:11, mass 0.141176996424; collision mesh filename=package://abby_urdf/caster_ipt_ca03a3d7.STL scale=0.0254 0.0254 0.0254; visual mesh filename=package://abby_urdf/caster_ipt_ca03a3d7.STL scale=0.0254 0.0254 0.0254
- added link caster:12, mass 0.141176996424; collision mesh filename=package://abby_urdf/caster_ipt_ca03a3d7.STL scale=0.0254 0.0254 0.0254; visual mesh filename=package://abby_urdf/caster_ipt_ca03a3d7.STL scale=0.0254 0.0254 0.0254
- added link frame:11, mass 3.238400046; collision mesh filename=package://abby_urdf/frame_ipt_29593391.STL scale=0.0254 0.0254 0.0254; visual mesh filename=package://abby_urdf/frame_ipt_29593391.STL scale=0.0254 0.0254 0.0254
- added link motor:11, mass 8.845051215; collision mesh filename=package://abby_urdf/motor_ipt_8185475f.STL scale=0.0254 0.0254 0.0254; visual mesh filename=package://abby_urdf/motor_ipt_8185475f.STL scale=0.0254 0.0254 0.0254
- added link motor_MIR:11, mass 2.88893887638; collision mesh filename=package://abby_urdf/motor_MIR_ipt_80c03f9e.STL scale=0.0254 0.0254 0.0254; visual mesh filename=package://abby_urdf/motor_MIR_ipt_80c03f9e.STL scale=0.0254 0.0254 0.0254
- added link wheel:11, mass 3.52668067675; collision mesh filename=package://abby_urdf/wheel_ipt_982fa4fe.STL scale=0.0254 0.0254 0.0254; visual mesh filename=package://abby_urdf/wheel_ipt_982fa4fe.STL scale=0.0254 0.0254 0.0254
- added link wheel:21, mass 3.52668067675; collision mesh filename=package://abby_urdf/wheel_ipt_982fa4fe.STL scale=0.0254 0.0254 0.0254; visual mesh filename=package://abby_urdf/wheel_ipt_982fa4fe.STL scale=0.0254 0.0254 0.0254
- link Breaker:11: mass 0.455268555 -> 0.0936536702263; geometry collision mesh filename=package://abby_urdf/Breaker_iam_746c8f85.STL scale=0.0254 0.0254 0.0254; visual mesh filename=package://abby_urdf/Breaker_iam_746c8f85.STL scale=0.0254 0.0254 0.0254
- link IRB120_Base_rev0:11: mass 30.212469 -> 6.21503193527; geometry collision mesh filename=package://abby_urdf/IRB120_Base_rev0_iam_38446303.STL scale=0.0254 0.0254 0.0254; visual mesh filename=package://abby_urdf/IRB120_Base_rev0_iam_38446303.STL scale=0.0254 0.0254 0.0254
- link IRB120_Link1_rev0:11: mass 14.91106995 -> 3.06736850696; geometry collision mesh filename=package://abby_urdf/IRB120_Link1_rev0_iam_3fe6e7e5.STL scale=0.0254 0.0254 0.0254; visual mesh filename=package://abby_urdf/IRB120_Link1_rev0_iam_3fe6e7e5.STL scale=0.0254 0.0254 0.0254
- link IRB120_Link2_rev0:11: mass 19.0011906 -> 3.90875060185; geometry collision mesh filename=package://abby_urdf/IRB120_Link2_rev0_iam_90725b7e.STL scale=0.0254 0.0254 0.0254; visual mesh filename=package://abby_urdf/IRB120_Link2_rev0_iam_90725b7e.STL scale=0.0254 0.0254 0.0254
- link IRB120_Link3_rev0:11: mass 14.3105382 -> 2.94383262499; geometry collision mesh filename=package://abby_urdf/IRB120_Link3_rev0_iam_86ced70a.STL scale=0.0254 0.0254 0.0254; visual mesh filename=package://abby_urdf/IRB120_Link3_rev0_iam_86ced70a.STL scale=0.0254 0.0254 0.0254
- link IRB120_Link4_rev0:11: mass 6.45520365 -> 1.32790527095; geometry collision mesh filename=package://abby_urdf/IRB120_Link4_rev0_iam_467bed4b.STL scale=0.0254 0.0254 0.0254; visual mesh filename=package://abby_urdf/IRB120_Link4_rev0_iam_467bed4b.STL scale=0.0254 0.0254 0.0254
- link IRB120_Link5_rev0:11: mass 2.6572896 -> 0.546633236934; geometry collision mesh filename=package://abby_urdf/IRB120_Link5_rev0_iam_8f44ede8.STL scale=0.0254 0.0254 0.0254; visual mesh filename=package://abby_urdf/IRB120_Link5_rev0_iam_8f44ede8.STL scale=0.0254 0.0254 0.0254
- link IRB120_Link6_rev0:11: mass 0.066493539 -> 0.0136784407912; geometry collision mesh filename=package://abby_urdf/IRB120_Link6_rev0_ipt_8026fdc3.STL scale=0.0254 0.0254 0.0254; visual mesh filename=package://abby_urdf/IRB120_Link6_rev0_ipt_8026fdc3.STL scale=0.0254 0.0254 0.0254
- link IRC5_Compact:11: mass 138.2535 -> 28.440241599; geometry collision mesh filename=package://abby_urdf/IRC5_Compact_ipt_c844072c.STL scale=0.0254 0.0254 0.0254; visual mesh filename=package://abby_urdf/IRC5_Compact_ipt_c844072c.STL scale=0.0254 0.0254 0.0254
- link Kinect:11: mass 3.49291845 -> 0.718531137393; geometry collision mesh filename=package://abby_urdf/Kinect_ipt_94e5d325.STL scale=0.0254 0.0254 0.0254; visual mesh filename=package://abby_urdf/Kinect_ipt_94e5d325.STL scale=0.0254 0.0254 0.0254
- link LIDAR Bracket:11: mass 0.81895905 -> 0.168468742142; geometry collision mesh filename=package://abby_urdf/LIDAR Bracket_ipt_795304a8.STL scale=0.0254 0.0254 0.0254; visual mesh filename=package://abby_urdf/LIDAR Bracket_ipt_795304a8.STL scale=0.0254 0.0254 0.0254
- link LIDAR PSU:11: mass 1.819125 -> 0.37421370525; geometry collision mesh filename=package://abby_urdf/LIDAR PSU_ipt_2888cf41.STL scale=0.0254 0.0254 0.0254; visual mesh filename=package://abby_urdf/LIDAR PSU_ipt_2888cf41.STL scale=0.0254 0.0254 0.0254
- link PC:11: mass 63.5827185 -> 13.0796535036; geometry collision mesh filename=package://abby_urdf/PC_ipt_a7ade237.STL scale=0.0254 0.0254 0.0254; visual mesh filename=package://abby_urdf/PC_ipt_a7ade237.STL scale=0.0254 0.0254 0.0254
- link SICK LMS291:11: mass 18.07087905 -> 3.71737544502; geometry collision mesh filename=package://abby_urdf/SICK LMS291_ipt_2ad4e53c.STL scale=0.0254 0.0254 0.0254; visual mesh filename=package://abby_urdf/SICK LMS291_ipt_2ad4e53c.STL scale=0.0254 0.0254 0.0254
- link Spike H:11: mass 0.124133121 -> 0.02553552678; geometry collision mesh filename=package://abby_urdf/Spike H_iam_f19c9874.STL scale=0.0254 0.0254 0.0254; visual mesh filename=package://abby_urdf/Spike H_iam_f19c9874.STL scale=0.0254 0.0254 0.0254
- link aim rail cross brace:11: mass 0.801272745 -> 0.164830477742; geometry collision mesh filename=package://abby_urdf/aim rail cross brace_ipt_926bd022.STL scale=0.0254 0.0254 0.0254; visual mesh filename=package://abby_urdf/aim rail cross brace_ipt_926bd022.STL scale=0.0254 0.0254 0.0254
- link arm rail:11: mass 8.9185194 -> 1.83463598709; geometry collision mesh filename=package://abby_urdf/arm rail_ipt_926bd022.STL scale=0.0254 0.0254 0.0254; visual mesh filename=package://abby_urdf/arm rail_ipt_926bd022.STL scale=0.0254 0.0254 0.0254
- link arm rail:21: mass 8.9185194 -> 1.83463598709; geometry collision mesh filename=package://abby_urdf/arm rail_ipt_926bd022.STL scale=0.0254 0.0254 0.0254; visual mesh filename=package://abby_urdf/arm rail_ipt_926bd022.STL scale=0.0254 0.0254 0.0254
- link back frame plate:11: mass 0.47233305 -> 0.0971640215777; geometry collision mesh filename=package://abby_urdf/back frame plate_ipt_475e4947.STL scale=0.0254 0.0254 0.0254; visual mesh filename=package://abby_urdf/back frame plate_ipt_475e4947.STL scale=0.0254 0.0254 0.0254
- link back frame plate:21: mass 0.47233305 -> 0.0971640215777; geometry collision mesh filename=package://abby_urdf/back frame plate_ipt_475e4947.STL scale=0.0254 0.0254 0.0254; visual mesh filename=package://abby_urdf/back frame plate_ipt_475e4947.STL scale=0.0254 0.0254 0.0254
- link base plate:11: mass 49.0464765 -> 11.253309185; geometry collision mesh filename=package://abby_urdf/base plate_iam_348b8023.STL scale=0.0254 0.0254 0.0254; visual mesh filename=package://abby_urdf/base plate_iam_348b8023.STL scale=0.0254 0.0254 0.0254
- link compressor:11: mass 10.3359375 -> 2.12621423437; geometry collision mesh filename=package://abby_urdf/compressor_iam_e870b89.STL scale=0.0254 0.0254 0.0254; visual mesh filename=package://abby_urdf/compressor_iam_e870b89.STL scale=0.0254 0.0254 0.0254
- link frame bracket:11: mass 3.472875 -> 0.71440798275; geometry collision mesh filename=package://abby_urdf/frame bracket_ipt_f5a4f28d.STL scale=0.0254 0.0254 0.0254; visual mesh filename=package://abby_urdf/frame bracket_ipt_f5a4f28d.STL scale=0.0254 0.0254 0.0254
- link frame bracket:41: mass 3.472875 -> 0.71440798275; geometry collision mesh filename=package://abby_urdf/frame bracket_ipt_f5a4f28d.STL scale=0.0254 0.0254 0.0254; visual mesh filename=package://abby_urdf/frame bracket_ipt_f5a4f28d.STL scale=0.0254 0.0254 0.0254
- link front frame plate:11: mass 0.352841895 -> 0.072583397455; geometry collision mesh filename=package://abby_urdf/front frame plate_ipt_3e5bfe16.STL scale=0.0254 0.0254 0.0254; visual mesh filename=package://abby_urdf/front frame plate_ipt_3e5bfe16.STL scale=0.0254 0.0254 0.0254
- link front frame plate:21: mass 0.352841895 -> 0.072583397455; geometry collision mesh filename=package://abby_urdf/front frame plate_ipt_3e5bfe16.STL scale=0.0254 0.0254 0.0254; visual mesh filename=package://abby_urdf/front frame plate_ipt_3e5bfe16.STL scale=0.0254 0.0254 0.0254
- link front left plate:11: mass 1.15054695 -> 0.236679962742; geometry collision mesh filename=package://abby_urdf/front left plate_ipt_a8be7025.STL scale=0.0254 0.0254 0.0254; visual mesh filename=package://abby_urdf/front left plate_ipt_a8be7025.STL scale=0.0254 0.0254 0.0254
- link front right plate:11: mass 1.149883245 -> 0.236543431439; geometry collision mesh filename=package://abby_urdf/front right plate_ipt_a8be7025.STL scale=0.0254 0.0254 0.0254; visual mesh filename=package://abby_urdf/front right plate_ipt_a8be7025.STL scale=0.0254 0.0254 0.0254
- link front top side rail:11: mass 0.975463335 -> 0.200663367787; geometry collision mesh filename=package://abby_urdf/front top side rail_ipt_926bd022.STL scale=0.0254 0.0254 0.0254; visual mesh filename=package://abby_urdf/front top side rail_ipt_926bd022.STL scale=0.0254 0.0254 0.0254
- link front top side rail:21: mass 0.975463335 -> 0.200663367787; geometry collision mesh filename=package://abby_urdf/front top side rail_ipt_926bd022.STL scale=0.0254 0.0254 0.0254; visual mesh filename=package://abby_urdf/front top side rail_ipt_926bd022.STL scale=0.0254 0.0254 0.0254
- link front upright:11: mass 3.01928445 -> 0.621099496317; geometry collision mesh filename=package://abby_urdf/front upright_ipt_926bd022.STL scale=0.0254 0.0254 0.0254; visual mesh filename=package://abby_urdf/front upright_ipt_926bd022.STL scale=0.0254 0.0254 0.0254
- link front upright:21: mass 3.01928445 -> 0.621099496317; geometry collision mesh filename=package://abby_urdf/front upright_ipt_926bd022.STL scale=0.0254 0.0254 0.0254; visual mesh filename=package://abby_urdf/front upright_ipt_926bd022.STL scale=0.0254 0.0254 0.0254
- link lower front rail:31: mass 3.3373998 -> 0.686539267537; geometry collision mesh filename=package://abby_urdf/lower front rail_ipt_926bd022.STL scale=0.0254 0.0254 0.0254; visual mesh filename=package://abby_urdf/lower front rail_ipt_926bd022.STL scale=0.0254 0.0254 0.0254
- link lower front rail:41: mass 3.3373998 -> 0.686539267537; geometry collision mesh filename=package://abby_urdf/lower front rail_ipt_926bd022.STL scale=0.0254 0.0254 0.0254; visual mesh filename=package://abby_urdf/lower front rail_ipt_926bd022.STL scale=0.0254 0.0254 0.0254
- link lower front rail:51: mass 3.3373998 -> 0.686539267537; geometry collision mesh filename=package://abby_urdf/lower front rail_ipt_926bd022.STL scale=0.0254 0.0254 0.0254; visual mesh filename=package://abby_urdf/lower front rail_ipt_926bd022.STL scale=0.0254 0.0254 0.0254
- link lower side rail:11: mass 3.81828825 -> 0.785463227511; geometry collision mesh filename=package://abby_urdf/lower side rail_ipt_926bd022.STL scale=0.0254 0.0254 0.0254; visual mesh filename=package://abby_urdf/lower side rail_ipt_926bd022.STL scale=0.0254 0.0254 0.0254
- link lower side rail:21: mass 3.81828825 -> 0.785463227511; geometry collision mesh filename=package://abby_urdf/lower side rail_ipt_926bd022.STL scale=0.0254 0.0254 0.0254; visual mesh filename=package://abby_urdf/lower side rail_ipt_926bd022.STL scale=0.0254 0.0254 0.0254
- link lower side rail:31: mass 3.81828825 -> 0.785463227511; geometry collision mesh filename=package://abby_urdf/lower side rail_ipt_926bd022.STL scale=0.0254 0.0254 0.0254; visual mesh filename=package://abby_urdf/lower side rail_ipt_926bd022.STL scale=0.0254 0.0254 0.0254
- link lower side rail:41: mass 3.81828825 -> 0.785463227511; geometry collision mesh filename=package://abby_urdf/lower side rail_ipt_926bd022.STL scale=0.0254 0.0254 0.0254; visual mesh filename=package://abby_urdf/lower side rail_ipt_926bd022.STL scale=0.0254 0.0254 0.0254
- link lower vertical rail:11: mass 2.6309619 -> 0.541217344037; geometry collision mesh filename=package://abby_urdf/lower vertical rail_ipt_926bd022.STL scale=0.0254 0.0254 0.0254; visual mesh filename=package://abby_urdf/lower vertical rail_ipt_926bd022.STL scale=0.0254 0.0254 0.0254
- link lower vertical rail:21: mass 2.6309619 -> 0.541217344037; geometry collision mesh filename=package://abby_urdf/lower vertical rail_ipt_926bd022.STL scale=0.0254 0.0254 0.0254; visual mesh filename=package://abby_urdf/lower vertical rail_ipt_926bd022.STL scale=0.0254 0.0254 0.0254
- link router keepout:11: mass 1.378125 -> 0.28349523125; geometry collision mesh filename=package://abby_urdf/router keepout_ipt_2b3ba7b4.STL scale=0.0254 0.0254 0.0254; visual mesh filename=package://abby_urdf/router keepout_ipt_2b3ba7b4.STL scale=0.0254 0.0254 0.0254
- link short frame bracket:11: mass 3.472875 -> 0.71440798275; geometry collision mesh filename=package://abby_urdf/short frame bracket_ipt_f5a4f28d.STL scale=0.0254 0.0254 0.0254; visual mesh filename=package://abby_urdf/short frame bracket_ipt_f5a4f28d.STL scale=0.0254 0.0254 0.0254
- link short frame bracket:21: mass 3.472875 -> 0.71440798275; geometry collision mesh filename=package://abby_urdf/short frame bracket_ipt_f5a4f28d.STL scale=0.0254 0.0254 0.0254; visual mesh filename=package://abby_urdf/short frame bracket_ipt_f5a4f28d.STL scale=0.0254 0.0254 0.0254
- link top plate:11: mass 11.7595296 -> 2.41906254029; geometry collision mesh filename=package://abby_urdf/top plate_ipt_9041f1eb.STL scale=0.0254 0.0254 0.0254; visual mesh filename=package://abby_urdf/top plate_ipt_9041f1eb.STL scale=0.0254 0.0254 0.0254
Joints:
- removed joint IRB120_Base_rev0:1--IRB120_Link1_rev0:11
- removed joint IRB120_Link2_rev0:1--IRB120_Link1_rev0:11
- removed joint IRB120_Link3_rev0:1--IRB120_Link2_rev0:11
- removed joint IRB120_Link3_rev0:1--IRB120_Link4_rev0:11
- removed joint IRB120_Link4_rev0:1--IRB120_Link5_rev0:11
- removed joint IRB120_Link5_rev0:1--IRB120_Link6_rev0:11
- removed joint back frame plate:1--invacare assy:11
- removed joint frame bracket:1--invacare assy:11
- removed joint frame bracket:11--base_link
- removed joint front frame plate:1--invacare assy:11
- removed joint invacare assy:1--back frame plate:21
- removed joint lower front rail:3--arm rail:21
- removed joint lower front rail:3--lower side rail:11
- removed joint lower front rail:5--short frame bracket:11
- removed joint router keepout:1--arm rail:21
- removed joint short frame bracket:2--invacare assy:11
- added joint ABB Base Joint: type revolute, parent IRB120_Base_rev0:11, child IRB120_Link1_rev0:11, origin xyz=0.04203954 0.09686036 8.01624008326e-05 rpy=-3.14159265359 -0.668845740547 3.14159265359, axis 0 1 0, limit lower=-3.141592 upper=3.141592 effort=300 velocity=10.0
- added joint ABB Fifth Joint: type revolute, parent IRB120_Link5_rev0:11, child IRB120_Link6_rev0:11, origin xyz=0.072000865279 7.81392714644e-07 -0.0620001796247 rpy=-1.5707961734 0.571193670262 -1.57079621992, axis 0 0 1, limit lower=-3.141592 upper=3.141592 effort=300 velocity=10.0
- added joint ABB First Joint: type revolute, parent IRB120_Link1_rev0:11, child IRB120_Link2_rev0:11, origin xyz=5.57577729543e-07 0.1134999 -0.0574996276953 rpy=-3.80159157889e-07 -2.82044180378e-07 1.9676191066, axis 0 0 1, limit lower=-3.141592 upper=0.0 effort=300 velocity=10.0
- added joint ABB Fourth Joint: type revolute, parent IRB120_Link4_rev0:11, child IRB120_Link5_rev0:11, origin xyz=500.302186066 0.00151566707848 0.0616850168905 rpy=1.62064242872e-07 3.95710603931e-07 -0.163660073928, axis 0 0 1, limit lower=-2.0 upper=2.0 effort=300 velocity=10.0
- added joint ABB Second Joint: type revolute, parent IRB120_Link2_rev0:11, child IRB120_Link3_rev0:11, origin xyz=1.65908264504e-06 0.270000153642 -0.00150067174086 rpy=3.2758892825e-07 1.65717751769e-07 0.989050240485, axis 0 0 1, limit lower=-2.141592 upper=1.0 effort=300 velocity=10.0
- added joint ABB Third Joint: type revolute, parent IRB120_Link3_rev0:11, child IRB120_Link4_rev0:11, origin xyz=-500.000188071 0.0701403024607 0.060593734446 rpy=-1.52544583094 1.29532332074e-07 2.10681567879e-07, axis 1 0 0, limit lower=-3.141592 upper=3.141592 effort=300 velocity=10.0
- added joint Left Caster: type continuous, parent frame:11, child caster:11, origin xyz=0.438376314 -0.0930717791273 -0.0402738600969 rpy=-0.113808556509 0.599759885216 -0.0644280863472, axis 0 1 0
- added joint Left Caster Wheel: type continuous, parent caster:11, child caster wheel:11, origin xyz=-0.0374391391943 -0.136525 0.057149470843 rpy=-4.13084785385e-07 0 1.57079632679, axis 0 1 0
- added joint Left Wheel: type continuous, parent motor_MIR:11, child wheel:11, origin xyz=0.156311015806 0.278257 -0.0913293179601 rpy=3.14159265359 0.902962593822 0, axis 0 1 0
- added joint Right Caster: type continuous, parent frame:11, child caster:12, origin xyz=0.007998714 -0.0930717791273 -0.0402738600969 rpy=-0.393667317717 1.32390459026 -0.382877964465, axis 0 1 0
- added joint Right Caster Wheel: type continuous, parent caster:12, child caster wheel:12, origin xyz=-0.0374398564987 -0.136525 0.0571499693664 rpy=-3.1415922422 -0.131082218832 -1.57079652096, axis 0 1 0
- added joint Right Wheel: type continuous, parent motor:11, child wheel:21, origin xyz=0.0494411886234 0.5008626 0.0986537374286 rpy=3.14159265359 -1.17052308335 0, axis 0 1 0
- added joint arm rail:2--front top side rail:11: type fixed, parent front top side rail:11, child arm rail:21, origin xyz=0.133350000005 0.0122885199645 0.96420432 rpy=0 1.57079632679 0
- added joint back frame plate:1--frame:11: type fixed, parent frame:11, child back frame plate:11, origin xyz=0.451495668 -0.00634752228531 -0.632080945917 rpy=1.5707959168 0 -3.14159265357
- added joint battery rails:1--motor_MIR:11: type fixed, parent battery rails:11, child motor_MIR:11, origin xyz=0 -0.0104648 -0.191353694 rpy=-3.14159265359 0.211571921606 -1.57079632679
- added joint battery:1--battery rails:11: type fixed, parent battery rails:11, child battery:11, origin xyz=0 -0.0118999 -0.34100008 rpy=0 0 0
- added joint battery:2--battery rails:11: type fixed, parent battery rails:11, child battery:21, origin xyz=0 -0.0388874 0.03999992 rpy=3.14159265359 0 3.14159265359
- added joint frame bracket:1--frame:11: type fixed, parent frame bracket:11, child frame:11, origin xyz=-0.0163353016417 0.217135176601 -0.44243540602 rpy=1.5707959168 0 -1.5707963268
- added joint frame:1--back frame plate:21: type fixed, parent frame:11, child back frame plate:21, origin xyz=0.428673514 -0.0063499370587 -0.689873885703 rpy=1.57079673678 0 0
- added joint frame:1--battery rails:11: type fixed, parent frame:11, child battery rails:11, origin xyz=0.223187514 -0.0365116467139 -0.661299066183 rpy=-3.04771179927 0 3.14159265359
- added joint front frame plate:1--frame:11: type fixed, parent frame:11, child front frame plate:11, origin xyz=0.45466 -0.00634840638155 -0.076202062522 rpy=-1.57079673678 0 3.14159265359
- added joint lower side rail:1--lower front rail:51: type fixed, parent lower side rail:11, child lower front rail:51, origin xyz=0 -0.0141996159995 -0.26619708 rpy=0 0 -1.57079632705
- added joint lower side rail:2--lower side rail:11: type fixed, parent lower side rail:21, child lower side rail:11, origin xyz=0 0 0 rpy=0 0 0
- added joint motor_MIR:1--motor:11: type fixed, parent motor_MIR:11, child motor:11, origin xyz=0.106869827183 0.2226056 0.00732441946858 rpy=3.14159265359 0 0
- added joint router keepout:1--top plate:11: type fixed, parent top plate:11, child router keepout:11, origin xyz=0.0848749280385 0.263535160001 -0.31115 rpy=1.57079632679 0 0
- added joint short frame bracket:2--frame:11: type fixed, parent frame:11, child short frame bracket:21, origin xyz=0.445437514 0 -0.689873906859 rpy=0.000140706182803 1.5707959168 1.57093703311
- joint IRB120_Base_rev0:1--arm rail:11: origin xyz=0.55055262 -0.0796391599982 0.2324448234 rpy=0 0 -3.14159265359 -> xyz=0.37592762 -0.0796391599982 0.2324448234 rpy=0 0 3.14159265359
- joint IRC5_Compact:1--lower vertical rail:21: origin xyz=-0.27484578 -0.52197457201 0.0408498038687 rpy=1.57095443956 1.57079632679 0.000126494212215 -> xyz=-0.27484578 -0.52197457201 0.0408498038687 rpy=1.57089118845 1.57079632679 0
- joint base plate:1--lower front rail:31: origin xyz=0.466924898 0.00750061999634 -0.00499872000083 rpy=0 0 1.57079632679 -> xyz=0.466924898 0.00750061999635 -0.00499872000083 rpy=0 0 1.57079632679
- joint compressor:1--top plate:11: origin xyz=0.174625066039 0.161925000001 -0.00634999999969 rpy=-1.57079632679 1.57079632679 6.32411066351e-05 -> xyz=0.174625066039 0.161925000001 -0.00634999999969 rpy=-1.5708595819 1.57079632679 0
- joint frame bracket:1--front upright:11: origin xyz=-0.605070815547 0.227632514004 0.445910562843 rpy=-1.5707963268 1.47691506249 3.14159265359 -> xyz=0.0472087385903 0.2215801766 -0.382035463768 rpy=-1.5707963268 1.47691506249 -3.14159265359
- joint frame bracket:4--frame bracket:11: origin xyz=-0.617813733008 -0.218772485996 0.391860873726 rpy=0 0 0 -> xyz=0.0344658211298 -0.2248248234 -0.436085152885 rpy=0 0 0
- joint front frame plate:2--frame bracket:11: origin xyz=-0.59241441583 0.235887514004 0.385512358526 rpy=0 0 -1.57079632679 -> xyz=0.0598651383077 0.2298351766 -0.442433668085 rpy=0 0 -1.57079632679
- joint front left plate:1--front right plate:11: origin xyz=0.384175 0.0933500799993 0 rpy=3.14159265359 0 3.14159265359 -> xyz=0.384175 0.0933500799993 0 rpy=-3.14159265359 0 3.14159265359
- joint front right plate:1--LIDAR PSU:11: origin xyz=0.00252806199982 -0.00324104 -0.000792480000552 rpy=0 0 1.57160500763 -> xyz=0.00252806199982 -0.00324104 -0.000792480000551 rpy=0 0 1.57160500763
- joint front top side rail:1--front upright:11: origin xyz=-0.34790888 -0.00126492 0 rpy=-1.57085818898 -1.57079632654 1.57085818905 -> xyz=-0.34790888 -0.00126492 0 rpy=-1.57085818895 -1.57079632654 1.57085818902
- joint front top side rail:2--front top side rail:11: origin xyz=0.45085000001 0.03700017988 0.0142011399992 rpy=-3.14159265359 0 3.14159265334 -> xyz=0.45085000001 0.03700017988 0.0142011399992 rpy=3.14159265359 0 3.14159265334
- joint lower front rail:3--front upright:11: origin xyz=-0.07291324 0.01873504 0 rpy=-3.14159265316 -1.57079632679 3.14159265316 -> xyz=-0.07291324 0.01873504 0 rpy=-3.13327192996 -1.57079632679 3.13327192996
- joint lower front rail:4--lower vertical rail:11: origin xyz=0.354977700001 -0.00410717987564 -0.496237514 rpy=0 -1.57079632674 3.14159265359 -> xyz=0.354977700001 -0.00410717987564 -0.496237514 rpy=1.80907794896e-07 -1.57079632674 3.14159247268
