Commit message: URDF files are now good (although arm height is estimated.)

File: abby_description/urdf/abby.urdf (robot description, URDF)
Before this commit: robot robot_no_arm, 32 links, 31 joints
Joints:
- removed joint frame_solid:1--r_drive wheel1
- added joint l_drive_wheel_joint: type continuous, parent frame_solid:11, child l_drive_wheel1, origin xyz=0.0466801199851 -0.217162738547 0.147715939724 rpy=0 -0.119809660819 1.57079632679, axis 0 -1 0
- joint compressor--top_plate1: origin xyz=0.40450007998 0.426550996313 -0.00635023492284 rpy=2.35081473332e-05 1.5707959092 1.57081983534 -> xyz=0.40450007998 0.426550996313 -0.00635023492284 rpy=2.35090778551e-05 1.5707959092 1.57081983614
- joint l_caster_joint: axis 3.49916e-011 0.437253 -0.899338 -> 0 1 0
- joint l_caster_wheel_joint: axis 0.863101 0.454195 0.220827 -> 0 1 0; origin xyz=0.0374386651859 -0.136525432368 0.0571509283666 rpy=6.29554520149e-07 -0.0978245101151 -1.57079646214 -> xyz=0.0374386651859 -0.136525432368 0.0571509283666 rpy=6.29554520079e-07 -0.0978245101151 -1.57079646214
- joint r_caster_joint: axis 3.49916e-011 0.437253 -0.899338 -> 0 1 0
- joint r_caster_wheel_joint: axis -0.997921 0.0579676 0.0281835 -> 0 1 0; origin xyz=0.0374395826544 -0.13652471423 0.0571493788518 rpy=-2.44191411353e-07 0.632428512243 -1.570796684 -> xyz=0.0374395826544 -0.13652471423 0.0571493788518 rpy=-2.44191411285e-07 0.632428512243 -1.570796684
- joint r_drive_wheel_joint: axis 1 2.88933e-011 5.29561e-011 -> 0 1 0; child l_drive_wheel1 -> r_drive wheel1; origin xyz=0.0466801199851 -0.217162738547 0.147715939724 rpy=0 -0.119809660819 1.57079632679 -> xyz=-0.509833626015 -0.217162738527 0.147715939697 rpy=0 -0.443332433305 -1.57079632679
- joint top_plate--spike_relay1: origin xyz=0.229875079988 0.264625478066 -0.00635030519038 rpy=3.14159264636 0 0.00520380555278 -> xyz=0.229875079988 0.264625478066 -0.00635030519039 rpy=3.14159264636 0 0.00520380555278

File: abby_description/urdf/abby.xacro (robot description, xacro)
@@ -1,685 +1,12 @@
 <?xml version="1.0" ?>
-<robot name="robot_no_arm" xmlns:xacro="http://ros.org/wiki/xacro">
+<robot name="abby" xmlns:xacro="http://ros.org/wiki/xacro">
 	<include filename="$(find abb_common)/urdf/irb_120_macro.xacro" />
+	<include filename="$(find abby_description)/urdf/abby_no_arm_macro.xacro" />
 	<xacro:irb_120 prefix="irb_120_"/>
+    <xacro:abby_no_arm />
     <joint name="frame_arm" type="fixed">
         <parent link="frame1"/>
         <child link="irb_120_base_link"/>
-		<origin rpy="3.1415926535 1.57079632679 0" xyz="0.046 -0.55 .75"/><!--xyz="0.243630043581 -0.0815492400606 0.0468452199958"/-->
+		<origin rpy="3.1415926535 1.57079632679 0" xyz="0.046 -0.55 .75"/>
     </joint>
-	<link name="frame1">
-		<visual>
-			<geometry>
-				<mesh filename="package://abby_description/meshes/al_frame_iam_3826baa4.stl" scale="0.0254 0.0254 0.0254"/>
-			</geometry>
-			<origin rpy="0 0 0" xyz="0.0446356739978 0.177065647653 -0.0893087163603"/>
-			<material name="frame1_color">
-				<color rgba="0.752941 0.752941 0.752941 1"/>
-			</material>
-		</visual>
-		<inertial>
-			<mass value="12.7774249075"/>
-			<inertia ixx="2.11995607184" ixy="-0.0128393605839" ixz="-0.0068818565379" iyy="1.84586933127" iyz="0.34872380742" izz="1.11710077832"/>
-			<origin rpy="0 0 0" xyz="0.0382793240557 -0.271251963735 0.649589084908"/>
-		</inertial>
-		<collision>
-			<geometry>
-				<mesh filename="package://abby_description/meshes/al_frame_iam_3826baa4.stl" scale="0.0254 0.0254 0.0254"/>
-			</geometry>
-			<origin rpy="0 0 0" xyz="0.0446356739978 0.177065647653 -0.0893087163603"/>
-		</collision>
-	</link>
-	<link name="f_r_frame_bracket1">
-		<visual>
-			<geometry>
-				<mesh filename="package://abby_description/meshes/frame bracket_ipt_f5a4f28d.stl" scale="0.0254 0.0254 0.0254"/>
-			</geometry>
-			<origin rpy="0 0 0" xyz="-0.0946635865578 -0.0205552039632 -0.424782665556"/>
-			<material name="f_r_frame_bracket1_color">
-				<color rgba="0.639216 0.639216 0.639216 1"/>
-			</material>
-		</visual>
-		<inertial>
-			<mass value="0.71440798275"/>
-			<inertia ixx="0.00043051877529" ixy="0.0" ixz="-1.18150140291e-05" iyy="0.00109167940213" iyz="0.0" izz="0.00105983757016"/>
-			<origin rpy="0 0 0" xyz="-0.0175668955453 0.00484479603152 -0.408054413923"/>
-		</inertial>
-		<collision>
-			<geometry>
-				<mesh filename="package://abby_description/meshes/frame bracket_ipt_f5a4f28d.stl" scale="0.0254 0.0254 0.0254"/>
-			</geometry>
-			<origin rpy="0 0 0" xyz="-0.0946635865578 -0.0205552039632 -0.424782665556"/>
-		</collision>
-	</link>
-	<joint name="frame--f_r_frame_bracket1" type="fixed">
-		<parent link="frame1"/>
-		<child link="f_r_frame_bracket1"/>
-		<origin rpy="0 -0.0938814541614 1.5707963268" xyz="-0.197196963951 -0.46840807491 0.660027160644"/>
-	</joint>
-	<link name="f_l_frame_bracket1">
-		<visual>
-			<geometry>
-				<mesh filename="package://abby_description/meshes/frame bracket_ipt_f5a4f28d.stl" scale="0.0254 0.0254 0.0254"/>
-			</geometry>
-			<origin rpy="0 0 0" xyz="-0.050800692836 -0.0508000000121 -0.00634958439213"/>
-			<material name="f_l_frame_bracket1_color">
-				<color rgba="0.639216 0.639216 0.639216 1"/>
-			</material>
-		</visual>
-		<inertial>
-			<mass value="0.71440798275"/>
-			<inertia ixx="0.00043051877529" ixy="0.0" ixz="-1.18150140291e-05" iyy="0.00109167940213" iyz="0.0" izz="0.00105983757016"/>
-			<origin rpy="0 0 0" xyz="0.026295998169 -0.025399999994 0.0103786672398"/>
-		</inertial>
-		<collision>
-			<geometry>
-				<mesh filename="package://abby_description/meshes/frame bracket_ipt_f5a4f28d.stl" scale="0.0254 0.0254 0.0254"/>
-			</geometry>
-			<origin rpy="0 0 0" xyz="-0.050800692836 -0.0508000000121 -0.00634958439213"/>
-		</collision>
-	</link>
-	<joint name="f_l_frame_bracket--f_r_frame_bracket1" type="fixed">
-		<parent link="f_r_frame_bracket1"/>
-		<child link="f_l_frame_bracket1"/>
-		<origin rpy="0 0 0" xyz="-0.0438628937327 -0.464082383966 -0.418433081198"/>
-	</joint>
-	<link name="f_l_frame_plate1">
-		<visual>
-			<geometry>
-				<mesh filename="package://abby_description/meshes/front frame plate_ipt_3e5bfe16.stl" scale="0.0254 0.0254 0.0254"/>
-			</geometry>
-			<origin rpy="0 0 0" xyz="0 0 0"/>
-			<material name="f_l_frame_plate1_color">
-				<color rgba="0.752941 0.752941 0.752941 1"/>
-			</material>
-		</visual>
-		<inertial>
-			<mass value="0.072583397455"/>
-			<inertia ixx="0.000139975007751" ixy="0.0" ixz="0.0" iyy="3.5475798236e-05" iyz="0.0" izz="0.000174962980108"/>
-			<origin rpy="0 0 0" xyz="0.0380034800186 0.0762017426097 0.00317605933453"/>
-		</inertial>
-		<collision>
-			<geometry>
-				<mesh filename="package://abby_description/meshes/front frame plate_ipt_3e5bfe16.stl" scale="0.0254 0.0254 0.0254"/>
-			</geometry>
-			<origin rpy="0 0 0" xyz="0 0 0"/>
-		</collision>
-	</link>
-	<joint name="f_l_frame_plate--f_l_frame_bracket1" type="fixed">
-		<parent link="f_l_frame_bracket1"/>
-		<child link="f_l_frame_plate1"/>
-		<origin rpy="-3.14159265359 0 1.57079632679" xyz="-0.050800692836 -0.0508000000121 -0.00634958439213"/>
-	</joint>
-	<link name="f_r_frame_plate1">
-		<visual>
-			<geometry>
-				<mesh filename="package://abby_description/meshes/front frame plate_ipt_3e5bfe16.stl" scale="0.0254 0.0254 0.0254"/>
-			</geometry>
-			<origin rpy="0 0 0" xyz="-0.0381000000045 -0.0762009322898 -0.00634941359797"/>
-			<material name="f_r_frame_plate1_color">
-				<color rgba="0.752941 0.752941 0.752941 1"/>
-			</material>
-		</visual>
-		<inertial>
-			<mass value="0.072583397455"/>
-			<inertia ixx="0.000139975007751" ixy="0.0" ixz="0.0" iyy="3.5475798236e-05" iyz="0.0" izz="0.000174962980108"/>
-			<origin rpy="0 0 0" xyz="-9.52500002381e-05 9.97890829413e-07 -0.00317559036918"/>
-		</inertial>
-		<collision>
-			<geometry>
-				<mesh filename="package://abby_description/meshes/front frame plate_ipt_3e5bfe16.stl" scale="0.0254 0.0254 0.0254"/>
-			</geometry>
-			<origin rpy="0 0 0" xyz="-0.0381000000045 -0.0762009322898 -0.00634941359797"/>
-		</collision>
-	</link>
-	<joint name="f_r_frame_plate--f_r_frame_bracket1" type="fixed">
-		<parent link="f_r_frame_bracket1"/>
-		<child link="f_r_frame_plate1"/>
-		<origin rpy="0 0 -1.57079632679" xyz="-0.0184628418291 -0.00785520396718 -0.424783134521"/>
-	</joint>
-	<link name="b_r_frame_bracket1">
-		<visual>
-			<geometry>
-				<mesh filename="package://abby_description/meshes/short frame bracket_ipt_f5a4f28d.stl" scale="0.0254 0.0254 0.0254"/>
-			</geometry>
-			<origin rpy="0 0 0" xyz="-0.0774480173821 -0.0263550400145 -0.00822489041407"/>
-			<material name="b_r_frame_bracket1_color">
-				<color rgba="0.639216 0.639216 0.639216 1"/>
-			</material>
-		</visual>
-		<inertial>
-			<mass value="0.71440798275"/>
-			<inertia ixx="0.00044432538895" ixy="0.0" ixz="-8.3387205787e-05" iyy="0.00086832128551" iyz="0.0" izz="0.00083243813657"/>
-			<origin rpy="0 0 0" xyz="-0.00691246125573 -0.000955040002614 0.00995368760594"/>
-		</inertial>
-		<collision>
-			<geometry>
-				<mesh filename="package://abby_description/meshes/short frame bracket_ipt_f5a4f28d.stl" scale="0.0254 0.0254 0.0254"/>
-			</geometry>
-			<origin rpy="0 0 0" xyz="-0.0774480173821 -0.0263550400145 -0.00822489041407"/>
-		</collision>
-	</link>
-	<joint name="frame--b_r_frame_bracket1" type="fixed">
-		<parent link="frame1"/>
-		<child link="b_r_frame_bracket1"/>
-		<origin rpy="0 -0.0938814541614 1.57079632654" xyz="-0.202996799965 0.113567247403 0.29642350598"/>
-	</joint>
-	<link name="b_r_frame_plate1">
-		<visual>
-			<geometry>
-				<mesh filename="package://abby_description/meshes/back frame plate_ipt_475e4947.stl" scale="0.0254 0.0254 0.0254"/>
-			</geometry>
-			<origin rpy="0 0 0" xyz="-0.0254000000255 -0.126998971214 1.58112569593e-06"/>
-			<material name="b_r_frame_plate1_color">
-				<color rgba="0.752941 0.752941 0.752941 1"/>
-			</material>
-		</visual>
-		<inertial>
-			<mass value="0.0971640215777"/>
-			<inertia ixx="0.0003344255636" ixy="8.4155085275e-07" ixz="0.0" iyy="4.7517225512e-05" iyz="0.0" izz="0.00038129137915"/>
-			<origin rpy="0 0 0" xyz="0.0126431039946 -0.025550836608 0.00317565745359"/>
-		</inertial>
-		<collision>
-			<geometry>
-				<mesh filename="package://abby_description/meshes/back frame plate_ipt_475e4947.stl" scale="0.0254 0.0254 0.0254"/>
-			</geometry>
-			<origin rpy="0 0 0" xyz="-0.0254000000255 -0.126998971214 1.58112569593e-06"/>
-		</collision>
-	</link>
-	<joint name="b_r_frame_plate--b_r_frame_bracket1" type="fixed">
-		<parent link="b_r_frame_bracket1"/>
-		<child link="b_r_frame_plate1"/>
-		<origin rpy="3.14159265359 0 -1.57079632679" xyz="-0.0520471238425 -0.000955040009423 -0.00822349691669"/>
-	</joint>
-	<link name="IRC5_Compact1">
-		<visual>
-			<geometry>
-				<mesh filename="package://abby_description/meshes/irc5_compact_ipt_c844072c.stl" scale="0.0254 0.0254 0.0254"/>
-			</geometry>
-			<origin rpy="0 0 0" xyz="-0.000849884100615 0.0283509919265 -0.462400284136"/>
-			<material name="IRC5_Compact1_color">
-				<color rgba="0.498039 0.498039 0.498039 1"/>
-			</material>
-		</visual>
-		<inertial>
-			<mass value="28.440241599"/>
-			<inertia ixx="0.75499468089" ixy="-0.00122306756239" ixz="-0.00124304296401" iyy="1.08063235538" iyz="-0.0064925615368" izz="0.61093241216"/>
-			<origin rpy="0 0 0" xyz="-0.225686620068 0.151686511222 -0.249482492333"/>
-		</inertial>
-		<collision>
-			<geometry>
-				<mesh filename="package://abby_description/meshes/irc5_compact_ipt_c844072c.stl" scale="0.0254 0.0254 0.0254"/>
-			</geometry>
-			<origin rpy="0 0 0" xyz="-0.000849884100615 0.0283509919265 -0.462400284136"/>
-		</collision>
-	</link>
-	<joint name="frame--IRC5_Compact1" type="fixed">
-		<parent link="frame1"/>
-		<child link="IRC5_Compact1"/>
-		<origin rpy="1.5707959092 0 3.14159265334" xyz="-0.18299683996 0.0935673788127 0.353829950251"/>
-	</joint>
-	<link name="router1">
-		<visual>
-			<geometry>
-				<mesh filename="package://abby_description/meshes/router keepout_ipt_2b3ba7b4.stl" scale="0.0254 0.0254 0.0254"/>
-			</geometry>
-			<origin rpy="0 0 0" xyz="0.0783000719655 0.725341498268 -1.11194969177e-06"/>
-			<material name="router1_color">
-				<color rgba="0.25098 0.321569 0.392157 1"/>
-			</material>
-		</visual>
-		<inertial>
-			<mass value="0.28349523125"/>
-			<inertia ixx="0.00067729370465" ixy="0.0" ixz="0.0" iyy="0.0008954399563" iyz="0.0" izz="0.00150414540089"/>
-			<origin rpy="0 0 0" xyz="0.0783000719663 0.727175853591 0.0190494073449"/>
-		</inertial>
-		<collision>
-			<geometry>
-				<mesh filename="package://abby_description/meshes/router keepout_ipt_2b3ba7b4.stl" scale="0.0254 0.0254 0.0254"/>
-			</geometry>
-			<origin rpy="0 0 0" xyz="0.0783000719655 0.725341498268 -1.11194969177e-06"/>
-		</collision>
-	</link>
-	<joint name="frame--router1" type="fixed">
-		<parent link="frame1"/>
-		<child link="router1"/>
-		<origin rpy="-1.5707959092 0 0" xyz="-0.0354469698523 -0.430316747951 1.61002981286"/>
-	</joint>
-	<link name="SICK_LMS2911">
-		<visual>
-			<geometry>
-				<mesh filename="package://abby_description/meshes/sick lms291_ipt_2ad4e53c.stl" scale="0.0254 0.0254 0.0254"/>
-			</geometry>
-			<origin rpy="0 0 0" xyz="-0.0683999139953 -0.00245779587475 -0.0929987962566"/>
-			<material name="SICK_LMS2911_color">
-				<color rgba="0.752941 0.752941 0.752941 1"/>
-			</material>
-		</visual>
-		<inertial>
-			<mass value="3.71737544502"/>
-			<inertia ixx="0.0174805834039" ixy="-4.4195210288e-07" ixz="4.1599227461e-07" iyy="0.0127643577208" iyz="0.00072853444335" izz="0.0175041992098"/>
-			<origin rpy="0 0 0" xyz="-0.0684016920036 0.0653465146418 -0.0708751847642"/>
-		</inertial>
-		<collision>
-			<geometry>
-				<mesh filename="package://abby_description/meshes/sick lms291_ipt_2ad4e53c.stl" scale="0.0254 0.0254 0.0254"/>
-			</geometry>
-			<origin rpy="0 0 0" xyz="-0.0683999139953 -0.00245779587475 -0.0929987962566"/>
-		</collision>
-	</link>
-	<joint name="frame--SICK_LMS2911" type="fixed">
-		<parent link="frame1"/>
-		<child link="SICK_LMS2911"/>
-		<origin rpy="1.5707959092 0 -3.14159265358" xyz="-0.0255468119868 -0.474758386705 0.311455920061"/>
-	</joint>
-	<link name="base_plate1">
-		<visual>
-			<geometry>
-				<mesh filename="package://abby_description/meshes/base plate_iam_348b8023.stl" scale="0.0254 0.0254 0.0254"/>
-			</geometry>
-			<origin rpy="0 0 0" xyz="-0.296284250178 -0.709693779926 -0.581261979343"/>
-			<material name="base_plate1_color">
-				<color rgba="0.752941 0.752941 0.752941 1"/>
-			</material>
-		</visual>
-		<inertial>
-			<mass value="11.253309185"/>
-			<inertia ixx="0.192702049774" ixy="-0.0128927375727" ixz="-0.00057983680454" iyy="0.235790506928" iyz="0.002976996201" izz="0.41200655867"/>
-			<origin rpy="0 0 0" xyz="-0.259429264405 -0.197794168785 -0.0311541484255"/>
-		</inertial>
-		<collision>
-			<geometry>
-				<mesh filename="package://abby_description/meshes/base plate_iam_348b8023.stl" scale="0.0254 0.0254 0.0254"/>
-			</geometry>
-			<origin rpy="0 0 0" xyz="-0.296284250178 -0.709693779926 -0.581261979343"/>
-		</collision>
-	</link>
-	<joint name="frame--base_plate1" type="fixed">
-		<parent link="frame1"/>
-		<child link="base_plate1"/>
-		<origin rpy="0 0 1.5707963268" xyz="-0.182996839959 0.0950674391444 0.365829741316"/>
-	</joint>
-	<link name="top_plate1">
-		<visual>
-			<geometry>
-				<mesh filename="package://abby_description/meshes/top plate_ipt_9041f1eb.stl" scale="0.0254 0.0254 0.0254"/>
-			</geometry>
-			<origin rpy="0 0 0" xyz="-0.039999919998 -0.0370003177082 -0.00635046315153"/>
-			<material name="top_plate1_color">
-				<color rgba="0.2 0.2 0.2 1"/>
-			</material>
-		</visual>
-		<inertial>
-			<mass value="2.41906254029"/>
-			<inertia ixx="0.070476646621" ixy="-3.2774173452e-05" ixz="0.0" iyy="0.05993791034" iyz="0.0" izz="0.130398461926"/>
-			<origin rpy="0 0 0" xyz="0.229580439988 0.257942378411 -0.00317445298106"/>
-		</inertial>
-		<collision>
-			<geometry>
-				<mesh filename="package://abby_description/meshes/top plate_ipt_9041f1eb.stl" scale="0.0254 0.0254 0.0254"/>
-			</geometry>
-			<origin rpy="0 0 0" xyz="-0.039999919998 -0.0370003177082 -0.00635046315153"/>
-		</collision>
-	</link>
-	<joint name="frame--top_plate1" type="fixed">
-		<parent link="frame1"/>
-		<child link="top_plate1"/>
-		<origin rpy="-3.14159265359 0 0" xyz="-0.182996839929 0.0965675138916 0.656087848989"/>
-	</joint>
-	<link name="main_breaker1">
-		<visual>
-			<geometry>
-				<mesh filename="package://abby_description/meshes/breaker_iam_746c8f85.stl" scale="0.0254 0.0254 0.0254"/>
-			</geometry>
-			<origin rpy="0 0 0" xyz="-0.0160837880011 -0.0289106364367 0.00508056290676"/>
-			<material name="main_breaker1_color">
-				<color rgba="0.752941 0.752941 0.752941 1"/>
-			</material>
-		</visual>
-		<inertial>
-			<mass value="0.0936536702263"/>
-			<inertia ixx="3.6925814571e-05" ixy="-4.3535021216e-06" ixz="1.05382973255e-07" iyy="2.44166070505e-05" iyz="-2.55254379072e-12" izz="4.8649438065e-05"/>
-			<origin rpy="0 0 0" xyz="-0.0161287460005 -0.0289109627394 0.0153385723229"/>
-		</inertial>
-		<collision>
-			<geometry>
-				<mesh filename="package://abby_description/meshes/breaker_iam_746c8f85.stl" scale="0.0254 0.0254 0.0254"/>
-			</geometry>
-			<origin rpy="0 0 0" xyz="-0.0160837880011 -0.0289106364367 0.00508056290676"/>
-		</collision>
-	</link>
-	<joint name="main_breaker--top_plate1" type="fixed">
-		<parent link="top_plate1"/>
-		<child link="main_breaker1"/>
-		<origin rpy="3.14159265359 0 0" xyz="0.426298867993 0.159767684312 -0.00635046455001"/>
-	</joint>
-	<link name="compressor1">
-		<visual>
-			<geometry>
-				<mesh filename="package://abby_description/meshes/compressor_iam_e870b89.stl" scale="0.0254 0.0254 0.0254"/>
-			</geometry>
-			<origin rpy="0 0 0" xyz="0.217095026073 0.0541649919903 0.058507418554"/>
-			<material name="compressor1_color">
-				<color rgba="0.752941 0.752941 0.752941 1"/>
-			</material>
-		</visual>
-		<inertial>
-			<mass value="2.12621423437"/>
-			<inertia ixx="-0.0061140063136" ixy="0.0073422915937" ixz="0.0121866630191" iyy="-0.0247184035886" iyz="0.0043080263318" izz="-0.0223276763534"/>
-			<origin rpy="0 0 0" xyz="0.0555649192101 -0.000189230004887 -0.0360164073274"/>
-		</inertial>
-		<collision>
-			<geometry>
-				<mesh filename="package://abby_description/meshes/compressor_iam_e870b89.stl" scale="0.0254 0.0254 0.0254"/>
-			</geometry>
-			<origin rpy="0 0 0" xyz="0.217095026073 0.0541649919903 0.058507418554"/>
-		</collision>
-	</link>
-	<joint name="compressor--top_plate1" type="fixed">
-		<parent link="top_plate1"/>
-		<child link="compressor1"/>
-		<origin rpy="2.35081473332e-05 1.5707959092 1.57081983534" xyz="0.40450007998 0.426550996313 -0.00635023492284"/>
-	</joint>
-	<link name="PC1">
-		<visual>
-			<geometry>
-				<mesh filename="package://abby_description/meshes/pc_ipt_a7ade237.stl" scale="0.0254 0.0254 0.0254"/>
-			</geometry>
-			<origin rpy="0 0 0" xyz="0 -0.095249567657 -1.93835330509e-07"/>
-			<material name="PC1_color">
-				<color rgba="0 0 0 1"/>
-			</material>
-		</visual>
-		<inertial>
-			<mass value="13.0796535036"/>
-			<inertia ixx="0.199045542023" ixy="0.000104306361732" ixz="0.00061701926176" iyy="0.3078833877" iyz="0.000148148651798" izz="0.128774326576"/>
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
File: abby_description/urdf/abby_no_arm_macro.xacro (robot description, xacro)
@@ -1,4 +1,5 @@
 <?xml version="1.0" ?>
-<robot name="robot_no_arm">
+<robot xmlns:xacro="http://ros.org/wiki/xacro">
+	<xacro:macro name="abby_no_arm">
 	<link name="frame1">
 		<visual>
@@ -677,3 +678,4 @@
 		<origin rpy="0 -0.443332433305 -1.57079632679" xyz="-0.509833626015 -0.217162738527 0.147715939697"/>
 	</joint>
+  </xacro:macro>
 </robot>

Commit message: Updated abby's xacros and urdf to include the kinect.
So far, the kinect is in the wrong place, and I need to get
measurements from the CAD file to properly place it.

File: abby_description/urdf/abby.urdf (robot description, URDF)
Before this commit: robot abby, 32 links, 31 joints
Links:
- added link camera_depth_frame, mass 0.01
- added link camera_depth_optical_frame, mass 0.001
- added link camera_link, mass 0.01; collision box size=0.0730 .2760 0.0720; visual mesh filename=package://cwru_description/meshes/kinect.dae
- added link camera_rgb_frame, mass 0.001
- added link camera_rgb_optical_frame, mass 0.001
Joints:
- added joint base_camera_joint: type fixed, parent frame1, child camera_link, origin xyz=0 0 0 rpy=0 0.436331944 -1.570795
- added joint camera_depth_joint: type fixed, parent camera_link, child camera_depth_frame, origin xyz=0 0.018 0 rpy=0 0 0
- added joint camera_depth_optical_joint: type fixed, parent camera_depth_frame, child camera_depth_optical_frame, origin xyz=0 0 0 rpy=-1.570795 0 -1.570795
- added joint camera_rgb_joint: type fixed, parent camera_link, child camera_rgb_frame, origin xyz=0 -0.005 0 rpy=0 0 0
- added joint camera_rgb_optical_joint: type fixed, parent camera_rgb_frame, child camera_rgb_optical_frame, origin xyz=0 0 0 rpy=-1.570795 0 -1.570795

File: abby_description/urdf/abby_no_arm_macro.xacro (robot description, xacro)
@@ -1,6 +1,8 @@
 <?xml version="1.0" ?>
 <robot xmlns:xacro="http://ros.org/wiki/xacro">
+    <include filename="$(find cwru_description)/urdf/kinect.urdf.xacro"/>
 	<xacro:macro name="abby_no_arm">
-	<link name="frame1">
+	  <xacro:kinect xyz="0 0 0" rpy="0 0.436331944 -1.570795" parent_frame="frame1" />
+	  <link name="frame1">
 		<visual>
 			<geometry>
@@ -23,6 +25,6 @@
 			<origin rpy="0 0 0" xyz="0.0446356739978 0.177065647653 -0.0893087163603"/>
 		</collision>
-	</link>
-	<link name="f_r_frame_bracket1">
+	  </link>
+	  <link name="f_r_frame_bracket1">
 		<visual>
 			<geometry>
@@ -45,5 +47,5 @@
 			<origin rpy="0 0 0" xyz="-0.0946635865578 -0.0205552039632 -0.424782665556"/>
 		</collision>
-	</link>
+	  </link>
 	<joint name="frame--f_r_frame_bracket1" type="fixed">
 		<parent link="frame1"/>

Commit message: Reworked launch files and tweaked urdf/xacros.
Launch files now create static transforms for LIDAR and base frame.
URDF now has accurate kinect position.
Still to do:
* Get arm position more accurate.
* Center Kinect better (?)
* Get base_link transform height correct
* Check/fix LIDAR transform

File: abby_description/urdf/abby.urdf (robot description, URDF)
Before this commit: robot abby, 37 links, 36 joints
Joints:
- joint base_camera_joint: origin xyz=0 0 0 rpy=0 0.436331944 -1.570795 -> xyz=0.04464 -0.6357 1.491 rpy=0 0.436331944 -1.570795

File: abby_description/urdf/abby_no_arm_macro.xacro (robot description, xacro)
@@ -3,5 +3,5 @@
     <include filename="$(find cwru_description)/urdf/kinect.urdf.xacro"/>
 	<xacro:macro name="abby_no_arm">
-	  <xacro:kinect xyz="0.414 -0.217502 -1.661" rpy="0 0.436331944 -1.570795" parent_frame="frame1" />
+	  <xacro:kinect xyz="0.04464 -0.6357 1.491" rpy="0 0.436331944 -1.570795" parent_frame="frame1" />
 	  <link name="frame1">
 		<visual>
