Commit message: Finished sick LIDAR xacro.
The LIDAR is now loaded into the model with a xacro in the cwru_description.
The xacro macro includes the model and the tf for the LIDAR, which allows
the removal of the tf broadcaster from the launch file.

File: abby_description/urdf/abby.urdf (robot description, URDF)
Before this commit: robot abby, 37 links, 36 joints
Links:
- removed link SICK_LMS2911
- added link SICK_LMS291, mass 3.71737544502; collision mesh filename=package://cwru_description/meshes/sick_lms291.stl scale=0.0254 0.0254 0.0254; visual mesh filename=package://cwru_description/meshes/sick_lms291.stl scale=0.0254 0.0254 0.0254
- added link base_laser1_link, mass 0.01
Joints:
- removed joint frame--SICK_LMS2911
- added joint SICK_laser_frame_joint: type fixed, parent SICK_LMS291, child base_laser1_link, origin xyz=-0.0683999139953 0.035 -0.093 rpy=1.266 1.571 2.837
- added joint base_laser_joint: type fixed, parent frame1, child SICK_LMS291, origin xyz=-0.0255468119868 -0.474758386705 0.311455920061 rpy=1.5707959092 0 -3.14159265358

File: abby_description/urdf/abby_no_arm_macro.xacro (robot description, xacro)
@@ -2,6 +2,8 @@
 <robot xmlns:xacro="http://ros.org/wiki/xacro">
     <include filename="$(find cwru_description)/urdf/kinect.urdf.xacro"/>
+    <include filename="$(find cwru_description)/urdf/sick_LMS291.urdf.xacro"/>
 	<xacro:macro name="abby_no_arm">
 	  <xacro:kinect xyz="0.04464 -0.6357 1.491" rpy="0 0.436331944 -1.570795" parent_frame="frame1" />
+	  <xacro:SICK_LMS291 parent_frame="frame1" laser_frame="base_laser1_link" rpy="1.5707959092 0 -3.14159265358" xyz="-0.0255468119868 -0.474758386705 0.311455920061"/>
 	  <link name="frame1">
 		<visual>
@@ -242,31 +244,4 @@
 		<origin rpy="-1.5707959092 0 0" xyz="-0.0354469698523 -0.430316747951 1.61002981286"/>
 	</joint>
-	<link name="SICK_LMS2911">
-		<visual>
-			<geometry>
-				<mesh filename="package://abby_description/meshes/sick lms291_ipt_2ad4e53c.stl" scale="0.0254 0.0254 0.0254"/>
-			</geometry>
-			<origin rpy="0 0 0" xyz="-0.0683999139953 -0.00245779587475 -0.0929987962566"/>
-			<material name="SICK_LMS2911_color">
-				<color rgba="0.752941 0.752941 0.752941 1"/>
-			</material>
-		</visual>
-		<inertial>
-			<mass value="3.71737544502"/>
-			<inertia ixx="0.0174805834039" ixy="-4.4195210288e-07" ixz="4.1599227461e-07" iyy="0.0127643577208" iyz="0.00072853444335" izz="0.0175041992098"/>
-			<origin rpy="0 0 0" xyz="-0.0684016920036 0.0653465146418 -0.0708751847642"/>
-		</inertial>
-		<collision>
-			<geometry>
-				<mesh filename="package://abby_description/meshes/sick lms291_ipt_2ad4e53c.stl" scale="0.0254 0.0254 0.0254"/>
-			</geometry>
-			<origin rpy="0 0 0" xyz="-0.0683999139953 -0.00245779587475 -0.0929987962566"/>
-		</collision>
-	</link>
-	<joint name="frame--SICK_LMS2911" type="fixed">
-		<parent link="frame1"/>
-		<child link="SICK_LMS2911"/>
-		<origin rpy="1.5707959092 0 -3.14159265358" xyz="-0.0255468119868 -0.474758386705 0.311455920061"/>
-	</joint>
 	<link name="base_plate1">
 		<visual>

Commit message: Fixes kinect angle (it's close anyway) and changes real robot to default to true in abby.launch.

File: abby_description/urdf/abby.urdf (robot description, URDF)
Before this commit: robot abby, 38 links, 37 joints
Joints:
- joint base_camera_joint: origin xyz=0.04464 -0.6357 1.491 rpy=0 0.436331944 -1.570795 -> xyz=0.04464 -0.6357 1.491 rpy=0 0.9599 -1.570795

File: abby_description/urdf/abby_no_arm_macro.xacro (robot description, xacro)
@@ -4,5 +4,5 @@
     <include filename="$(find cwru_description)/urdf/sick_LMS291.urdf.xacro"/>
 	<xacro:macro name="abby_no_arm">
-	  <xacro:kinect xyz="0.04464 -0.6357 1.491" rpy="0 0.436331944 -1.570795" parent_frame="frame1" />
+	  <xacro:kinect xyz="0.04464 -0.6357 1.491" rpy="0 0.9599 -1.570795" parent_frame="frame1" />
 	  <xacro:SICK_LMS291 parent_frame="frame1" laser_frame="base_laser1_link" rpy="1.5707959092 0 -3.14159265358" xyz="-0.0255468119868 -0.474758386705 0.311455920061"/>
 	  <link name="frame1">

Commit message: Gripper defined in model.
Added gripper to abby's xacros and urdfs with correct measurements.
Added gripper joint state publisher to arduino node.

Arduino joint state publisher is tested and publishing correct
messages. Robot model appears properly in rviz.

File: abby_description/urdf/abby.urdf (robot description, URDF)
Before this commit: robot abby, 41 links, 40 joints
Joints:
- joint gripper__jaw_1: limit lower=-0.03175 upper=-0.022225 effort=1 velocity=1 -> lower=-0.039 upper=-0.03 effort=1 velocity=1; origin xyz=0 0 0.07699 rpy=0 0 3.14159265359 -> xyz=0 0 0.075 rpy=0 0 3.14159265359
- joint gripper_jaw_2: limit lower=-0.03175 upper=-0.022225 effort=1 velocity=1 -> lower=-0.039 upper=-0.03 effort=1 velocity=1; origin xyz=0 0 0.07699 rpy=0 0 0 -> xyz=0 0 0.075 rpy=0 0 0

File: abby_description/urdf/gripper.urdf (robot description, URDF)
Before this commit: robot abby, 41 links, 40 joints
Links:
- removed link IRC5_Compact1
- removed link PC1
- removed link SICK_LMS291
- removed link b_l_frame_bracket1
- removed link b_l_frame_plate1
- removed link b_r_frame_bracket1
- removed link b_r_frame_plate1
- removed link base_laser1_link
- removed link base_plate1
- removed link camera_depth_frame
- removed link camera_depth_optical_frame
- removed link camera_link
- removed link camera_rgb_frame
- removed link camera_rgb_optical_frame
- removed link compressor1
- removed link f_l_frame_bracket1
- removed link f_l_frame_plate1
- removed link f_r_frame_bracket1
- removed link f_r_frame_plate1
- removed link frame1
- removed link frame_solid:11
- removed link irb_120_base_link
- removed link irb_120_link_1
- removed link irb_120_link_2
- removed link irb_120_link_3
- removed link irb_120_link_4
- removed link irb_120_link_5
- removed link irb_120_link_6
- removed link l_caster1
- removed link l_caster_wheel1
- removed link l_drive_wheel1
- removed link main_breaker1
- removed link r_caster1
- removed link r_caster_wheel1
- removed link r_drive wheel1
- removed link router1
- removed link spike_relay1
- removed link top_plate1
Joints:
- removed joint PC--top_plate1
- removed joint SICK_laser_frame_joint
- removed joint arm_gripper
- removed joint b_l_frame_bracket--frame1
- removed joint b_l_frame_plate--b_l_frame_bracket1
- removed joint b_l_frame_plate--frame_solid:11
- removed joint b_r_frame_plate--b_r_frame_bracket1
- removed joint base_camera_joint
- removed joint base_laser_joint
- removed joint camera_depth_joint
- removed joint camera_depth_optical_joint
- removed joint camera_rgb_joint
- removed joint camera_rgb_optical_joint
- removed joint compressor--top_plate1
- removed joint f_l_frame_bracket--f_r_frame_bracket1
- removed joint f_l_frame_plate--f_l_frame_bracket1
- removed joint f_r_frame_plate--f_r_frame_bracket1
- removed joint frame--IRC5_Compact1
- removed joint frame--b_r_frame_bracket1
- removed joint frame--base_plate1
- removed joint frame--f_r_frame_bracket1
- removed joint frame--router1
- removed joint frame--top_plate1
- removed joint frame_arm
- removed joint joint1
- removed joint joint2
- removed joint joint3
- removed joint joint4
- removed joint joint5
- removed joint joint6
- removed joint l_caster_joint
- removed joint l_caster_wheel_joint
- removed joint l_drive_wheel_joint
- removed joint main_breaker--top_plate1
- removed joint r_caster_joint
- removed joint r_caster_wheel_joint
- removed joint r_drive_wheel_joint
- removed joint top_plate--spike_relay1
- joint gripper__jaw_1: limit lower=-0.03175 upper=-0.022225 effort=1 velocity=1 -> lower=-0.039 upper=-0.03 effort=1 velocity=1; origin xyz=0 0 0.07699 rpy=0 0 3.14159265359 -> xyz=0 0 0.075 rpy=0 0 3.14159265359
- joint gripper_jaw_2: limit lower=-0.03175 upper=-0.022225 effort=1 velocity=1 -> lower=-0.039 upper=-0.03 effort=1 velocity=1; origin xyz=0 0 0.07699 rpy=0 0 0 -> xyz=0 0 0.075 rpy=0 0 0

File: abby_description/urdf/gripper_macro.xacro (robot description, xacro)
@@ -71,12 +71,12 @@
 		<parent link="gripper_body"/>
 		<child link="gripper_jaw_1"/>
-		<origin rpy="0 0 3.14159265359" xyz="0 0 0.07699"/>
-		<limit upper="-0.022225" lower="-0.03175" effort="1" velocity="1" />
+		<origin rpy="0 0 3.14159265359" xyz="0 0 0.075"/>
+		<limit upper="-0.03" lower="-0.039" effort="1" velocity="1" />
 	</joint>
 	<joint name="gripper_jaw_2" type="prismatic">
 		<parent link="gripper_body"/>
 		<child link="gripper_jaw_2"/>
-		<origin rpy="0 0 0" xyz="0 0 0.07699"/>
-		<limit upper="-0.022225" lower="-0.03175" effort="1" velocity="1" />
+		<origin rpy="0 0 0" xyz="0 0 0.075"/>
+		<limit upper="-0.03" lower="-0.039" effort="1" velocity="1" />
 	</joint>
   </xacro:macro>

Commit message: Fixed a typo in the gripper description.

File: abby_description/urdf/abby.urdf (robot description, URDF)
Before this commit: robot abby, 41 links, 40 joints
Joints:
- removed joint gripper__jaw_1
- added joint gripper_jaw_1: type prismatic, parent gripper_body, child gripper_jaw_1, origin xyz=0 0 0.075 rpy=0 0 3.14159265359, limit lower=-0.039 upper=-0.03 effort=1 velocity=1

File: abby_description/urdf/gripper.urdf (robot description, URDF)
Before this commit: robot abby_gripper, 3 links, 2 joints
Joints:
- removed joint gripper__jaw_1
- added joint gripper_jaw_1: type prismatic, parent gripper_body, child gripper_jaw_1, origin xyz=0 0 0.075 rpy=0 0 3.14159265359, limit lower=-0.039 upper=-0.03 effort=1 velocity=1

File: abby_description/urdf/gripper_macro.xacro (robot description, xacro)
@@ -68,5 +68,5 @@
 		</collision>
 	</link>
-	<joint name="gripper__jaw_1" type="prismatic">
+	<joint name="gripper_jaw_1" type="prismatic">
 		<parent link="gripper_body"/>
 		<child link="gripper_jaw_1"/>

Commit message: Creates a script to move the arm to stow position.
The abby_arm_actions package will eventually contain an action server
to take commands such as "stow arm," "store object," etc. For now,
it has a script to stow the arm. This script should work, but the
arm navigation stack currently thinks it is in collision even when it
is not and refuses to plan a trajectory.

Also adds the stl file for the bin to the repository.

Also adds some launch files to the arm navigation package.

File: abby_description/urdf/abby.urdf (robot description, URDF)
Before this commit: robot abby, 41 links, 40 joints
Links:
- added link bin, mass 4.36697868587; collision mesh filename=package://abby_description/meshes/bin_ipt.stl scale=0.0254 0.0254 0.0254; visual mesh filename=package://abby_description/meshes/bin_ipt.stl scale=0.0254 0.0254 0.0254
Joints:
- added joint frame-bin: type fixed, parent frame1, child bin, origin xyz=-0.035 -0.474758386705 0.592669 rpy=1.57079619722 0 -1.57079632679

File: abby_description/urdf/abby_no_arm_macro.xacro (robot description, xacro)
@@ -654,5 +654,32 @@
         <axis xyz="0 1 0"/>
 		<origin rpy="0 -0.443332433305 -1.57079632679" xyz="-0.509833626015 -0.217162738527 0.147715939697"/>
-	</joint>
+    </joint>
+    <link name="bin">
+        <visual>
+            <geometry>
+                <mesh filename="package://abby_description/meshes/bin_ipt.stl" scale="0.0254 0.0254 0.0254"/>
+            </geometry>
+			<origin rpy="0 0 0" xyz="0 0 0"/>
+            <material name="yellow bin plastic">
+                <color rgba="0.98 0.98 0 1"/>
+            </material>
+        </visual>
+        <inertial>
+            <mass value="4.36697868587"/>
+			<inertia ixx="0.044427271429" ixy="0.00203259222186" ixz="-1.69295186692e-05" iyy="0.100418971824" iyz="3.3400709269e-06" izz="0.080242528585"/>
+			<origin rpy="0 0 0" xyz="0.17978882 -0.0977169394 0.104752255"/>
+		</inertial>
+        <collision>
+            <geometry>
+                <mesh filename="package://abby_description/meshes/bin_ipt.stl" scale="0.0254 0.0254 0.0254"/>
+            </geometry>
+			<origin rpy="0 0 0" xyz="0 0 0"/>
+        </collision>
+    </link>
+    <joint name="frame-bin" type="fixed">
+        <parent link="frame1"/>
+        <child link="bin"/>
+		<origin rpy="1.57079619722 0 -1.57079632679" xyz="-0.035 -0.474758386705 0.592669"/>
+    </joint>
   </xacro:macro>
 </robot>

Commit message: Kinect angle is now correct.
Kinect angle is set to ~51 degrees, which is accurate to less
than one degree, according to a plane fit of the floor from the
depth_registered point cloud.

File: abby_description/urdf/abby.urdf (robot description, URDF)
Before this commit: robot abby, 42 links, 41 joints
Joints:
- joint base_camera_joint: origin xyz=0.04464 -0.6357 1.491 rpy=0 0.9599 -1.570795 -> xyz=0.04464 -0.6357 1.491 rpy=0 0.8901 -1.570795

File: abby_description/urdf/abby_no_arm_macro.xacro (robot description, xacro)
@@ -4,5 +4,5 @@
     <include filename="$(find cwru_description)/urdf/sick_LMS291.urdf.xacro"/>
 	<xacro:macro name="abby_no_arm">
-	  <xacro:kinect xyz="0.04464 -0.6357 1.491" rpy="0 0.9599 -1.570795" parent_frame="frame1" />
+	  <xacro:kinect xyz="0.04464 -0.6357 1.491" rpy="0 0.8901 -1.570795" parent_frame="frame1" />
 	  <xacro:SICK_LMS291 parent_frame="frame1" laser_frame="base_laser1_link" rpy="1.5707959092 0 -3.14159265358" xyz="-0.0255468119868 -0.474758386705 0.311455920061"/>
 	  <link name="frame1">

Commit message: Kinect position is now correct.
Vertical translation and pitch rotation are correct (see previous commits).
Horizontal position is correct; agrees with LIDAR to <1cm.

File: abby_description/urdf/abby.urdf (robot description, URDF)
Before this commit: robot abby, 42 links, 41 joints
Joints:
- joint base_camera_joint: origin xyz=0.04464 -0.6357 1.491 rpy=0 0.8901 -1.570795 -> xyz=0.04464 -0.6557 1.491 rpy=0 0.8901 -1.570795

File: abby_description/urdf/abby_no_arm_macro.xacro (robot description, xacro)
@@ -4,5 +4,5 @@
     <include filename="$(find cwru_description)/urdf/sick_LMS291.urdf.xacro"/>
 	<xacro:macro name="abby_no_arm">
-	  <xacro:kinect xyz="0.04464 -0.6357 1.491" rpy="0 0.8901 -1.570795" parent_frame="frame1" />
+	  <xacro:kinect xyz="0.04464 -0.6557 1.491" rpy="0 0.8901 -1.570795" parent_frame="frame1" />
 	  <xacro:SICK_LMS291 parent_frame="frame1" laser_frame="base_laser1_link" rpy="1.5707959092 0 -3.14159265358" xyz="-0.0255468119868 -0.474758386705 0.311455920061"/>
 	  <link name="frame1">

Commit message: Fixes LIDAR definition and adds self filter.
LIDAR definition had the sensor frame off by about 6cm.
Also fixes abby's Kinect to match the corrected LIDAR frame.
Also adds self-filtering to the arm launch file.

File: abby_description/urdf/abby.urdf (robot description, URDF)
Before this commit: robot abby, 42 links, 41 joints
Joints:
- joint SICK_laser_frame_joint: origin xyz=-0.0683999139953 0.035 -0.093 rpy=1.266 1.571 2.837 -> xyz=-0.0683999139953 0.035 -0.0273 rpy=1.266 1.571 2.837
- joint base_camera_joint: origin xyz=0.04464 -0.6557 1.491 rpy=0 0.8901 -1.570795 -> xyz=0.04464 -0.59 1.491 rpy=0 0.8901 -1.570795

File: abby_description/urdf/abby_no_arm_macro.xacro (robot description, xacro)
@@ -4,5 +4,5 @@
     <include filename="$(find cwru_description)/urdf/sick_LMS291.urdf.xacro"/>
 	<xacro:macro name="abby_no_arm">
-	  <xacro:kinect xyz="0.04464 -0.6557 1.491" rpy="0 0.8901 -1.570795" parent_frame="frame1" />
+	  <xacro:kinect xyz="0.04464 -0.59 1.491" rpy="0 0.8901 -1.570795" parent_frame="frame1" />
 	  <xacro:SICK_LMS291 parent_frame="frame1" laser_frame="base_laser1_link" rpy="1.5707959092 0 -3.14159265358" xyz="-0.0255468119868 -0.474758386705 0.311455920061"/>
 	  <link name="frame1">

Commit message: Updated gripper to meshes and dimensions for acrylic plates.

File: abby_description/urdf/abby.urdf (robot description, URDF)
Before this commit: robot abby, 42 links, 41 joints
Joints:
- joint gripper_jaw_1: origin xyz=0 0 0.075 rpy=0 0 3.14159265359 -> xyz=0 0 0.062 rpy=0 0 3.14159265359
- joint gripper_jaw_2: origin xyz=0 0 0.075 rpy=0 0 0 -> xyz=0 0 0.062 rpy=0 0 0

File: abby_description/urdf/gripper_macro.xacro (robot description, xacro)
@@ -7,5 +7,5 @@
 				<mesh filename="package://abby_description/meshes/gripper_body.stl" scale="0.0254 0.0254 0.0254"/>
 			</geometry>
-			<origin rpy="3.141592653 0 0" xyz="0 0 0.02497074"/>
+			<origin rpy="3.141592653 0 0" xyz="0 0 0.012"/>
 			<material name="gripper:21_color">
 				<color rgba="0.752941 0.752941 0.752941 1"/>
@@ -21,5 +21,5 @@
 				<mesh filename="package://abby_description/meshes/gripper_body.stl" scale="0.0254 0.0254 0.0254"/>
 			</geometry>
-			<origin rpy="3.141592653 0 0" xyz="0 0 0.02497074"/>
+			<origin rpy="3.141592653 0 0" xyz="0 0 0.012"/>
 		</collision>
 	</link>
@@ -71,5 +71,5 @@
 		<parent link="gripper_body"/>
 		<child link="gripper_jaw_1"/>
-		<origin rpy="0 0 3.14159265359" xyz="0 0 0.075"/>
+		<origin rpy="0 0 3.14159265359" xyz="0 0 0.062"/>
 		<limit upper="-0.03" lower="-0.039" effort="1" velocity="1" />
 	</joint>
@@ -77,5 +77,5 @@
 		<parent link="gripper_body"/>
 		<child link="gripper_jaw_2"/>
-		<origin rpy="0 0 0" xyz="0 0 0.075"/>
+		<origin rpy="0 0 0" xyz="0 0 0.062"/>
 		<limit upper="-0.03" lower="-0.039" effort="1" velocity="1" />
 	</joint>

Commit message: Updated joint limits on arm.

File: abby_description/urdf/abby.urdf (robot description, URDF)
Before this commit: robot abby, 42 links, 41 joints
Joints:
- joint joint3: limit lower=-1.92 upper=1.22 effort=300 velocity=4.36 -> lower=-1.575 upper=1.23 effort=300 velocity=4.36
- joint joint4: limit lower=-2.79 upper=2.79 effort=300 velocity=5.58 -> lower=-2.80 upper=2.80 effort=300 velocity=5.58
- joint joint5: limit lower=-2.09 upper=2.09 effort=300 velocity=5.58 -> lower=-2.10 upper=2.10 effort=300 velocity=5.58
- joint joint6: limit lower=-6.98 upper=6.98 effort=300 velocity=7.33 -> lower=-6.985 upper=6.985 effort=300 velocity=7.33

Commit message: Fixes gripper origin.
Still need to get gripper rotation right.

File: abby_description/urdf/abby.urdf (robot description, URDF)
Before this commit: robot abby, 42 links, 41 joints
Joints:
- joint joint4: origin xyz=-500.000188071 0.0701403024607 0.060593734446 rpy=0 0 0 -> xyz=-0.000188071 0.0701403024607 0.060593734446 rpy=0 0 0
- joint joint5: origin xyz=500.302186066 0.00151566707848 0.0616850168905 rpy=0 0 0 -> xyz=0.302186066 0.00151566707848 0.0616850168905 rpy=0 0 0

File: abby_description/urdf/gripper_macro.xacro (robot description, xacro)
@@ -7,5 +7,5 @@
 				<mesh filename="package://abby_description/meshes/gripper_body.stl" scale="0.0254 0.0254 0.0254"/>
 			</geometry>
-			<origin rpy="3.141592653 0 0" xyz="0 0 0.012"/>
+			<origin rpy="3.141592653 0 0" xyz="0 0 0.017"/>
 			<material name="gripper:21_color">
 				<color rgba="0.752941 0.752941 0.752941 1"/>
@@ -15,5 +15,5 @@
 			<mass value="0.222800943405"/>
 			<inertia ixx="0.000113884956016" ixy="0.0" ixz="0.0" iyy="0.000132512764251" iyz="-4.2661207134e-07" izz="9.078477651e-05"/>
-			<origin rpy="3.141592653 0 0" xyz="0 0 0.008255"/>
+			<origin rpy="3.141592653 0 0" xyz="0 0 0.013255"/>
 		</inertial>
 		<collision>
@@ -21,5 +21,5 @@
 				<mesh filename="package://abby_description/meshes/gripper_body.stl" scale="0.0254 0.0254 0.0254"/>
 			</geometry>
-			<origin rpy="3.141592653 0 0" xyz="0 0 0.012"/>
+			<origin rpy="3.141592653 0 0" xyz="0 0 0.017"/>
 		</collision>
 	</link>

Commit message: Fixed gripper position in URDF and XACRO.
Gripper orientation is now approximately correct.

Also created a utility to publish dummy gripper states.

File: abby_description/urdf/abby.urdf (robot description, URDF)
Before this commit: robot abby, 42 links, 41 joints
Joints:
- joint arm_gripper: origin xyz=0 0 0 rpy=0 0 0 -> xyz=0 0 0 rpy=0 0 -0.7

File: abby_description/urdf/abby.xacro (robot description, xacro)
@@ -15,5 +15,5 @@
         <parent link="irb_120_link_6"/>
         <child link="gripper_body"/>
-		<origin rpy="0 0 0" xyz="0 0 0"/>
+		<origin rpy="0 0 -0.7" xyz="0 0 0"/>
     </joint>
 </robot>

Commit message: Updated kinect macro.
Kinect optical frames are published by the camera driver, making the
optical frames in the URDF redundant. Moved these to a separate macro.

File: abby_description/urdf/abby.urdf (robot description, URDF)
Before this commit: robot abby, 42 links, 41 joints
Links:
- removed link camera_depth_frame
- removed link camera_depth_optical_frame
- removed link camera_rgb_frame
- removed link camera_rgb_optical_frame
Joints:
- removed joint camera_depth_joint
- removed joint camera_depth_optical_joint
- removed joint camera_rgb_joint
- removed joint camera_rgb_optical_joint
- joint joint4: origin xyz=-0.000188071 0.0701403024607 0.060593734446 rpy=0 0 0 -> xyz=-500.000188071 0.0701403024607 0.060593734446 rpy=0 0 0
- joint joint5: origin xyz=0.302186066 0.00151566707848 0.0616850168905 rpy=0 0 0 -> xyz=500.302186066 0.00151566707848 0.0616850168905 rpy=0 0 0

Commit message: Simplified IRB-120 joints and regenerated IK solver.
IRB-120 joints no longer have weird offsets that cancel each other
out, greatly simplifying the joint geometry. (See swri-ros-pkg commit
comments.)

Updated URDF and IK solver to match new joint geometry.

This has not been tested at this time.

File: abby_description/urdf/abby.urdf (robot description, URDF)
Before this commit: robot abby, 38 links, 37 joints
Links:
- link irb_120_base_link: mass 6.21503193527 -> None
- link irb_120_link_1: mass 3.06736850696 -> None
- link irb_120_link_2: mass 3.90875060185 -> None
- link irb_120_link_3: mass 2.94383262499 -> None
- link irb_120_link_4: mass 1.32790527095 -> None
- link irb_120_link_5: mass 0.546633236934 -> None
- link irb_120_link_6: mass 0.0136784407912 -> None
Joints:
- joint joint1: origin xyz=0.04203954 0.09686036 0 rpy=-3.14159265359 3.14159265359 3.14159265359 -> xyz=0 0 0 rpy=-3.14159265359 3.14159265359 3.14159265359
- joint joint2: origin xyz=0 0.1134999 0.0574996276953 rpy=3.14159265359 0 3.14159265359 -> xyz=0 0.290 0 rpy=3.14159265359 0 3.14159265359
- joint joint3: origin xyz=0 0.270000153642 0.108 rpy=3.14159265359 0 3.14159265359 -> xyz=0 0.270 0 rpy=3.14159265359 0 3.14159265359
- joint joint4: origin xyz=-500.000188071 0.0701403024607 0.060593734446 rpy=0 0 0 -> xyz=0 0.070 0 rpy=0 0 0
- joint joint5: origin xyz=500.302186066 0.00151566707848 0.0616850168905 rpy=0 0 0 -> xyz=0.302 0 0 rpy=0 0 0
- joint joint6: origin xyz=0.072000865279 0 -0.0620001796247 rpy=-1.5707961734 0 -1.57079621992 -> xyz=0.072 0 0 rpy=-1.5707961734 0 -1.57079621992
