Commit message: Added some kinect utitlities.

File: abby_description/urdf/abby_no_arm_macro.xacro (robot description, xacro)
@@ -682,4 +682,24 @@
 		<origin rpy="1.57079619722 0 -1.57079632679" xyz="-0.035 -0.474758386705 0.592669"/>
     </joint>
+    <link name="tanks">
+        <visual>
+            <geometry>
+                <cylinder radius="0.055" length="0.50" />
+            </geometry>
+			<material name="metal">
+				<color rgba="0.752941 0.752941 0.752941 1"/>
+            </material>
+        </visual>
+        <collision>
+            <geometry>
+                <cylinder radius="0.055" length="0.50" />
+            </geometry>
+        </collision>
+    </link>
+    <joint name="frame-tanks" type="fixed">
+        <parent link="frame1"/>
+        <child link="tanks"/>
+		<origin rpy="0 0 0" xyz="0.03 -0.4 0.7"/>
+    </joint>
   </xacro:macro>
 </robot>

Commit message: Adds air tanks and warning light.
Air tank and warning light are in the model as simple cylinders.
This should prevent the robot from colliding with them.

File: abby_description/urdf/abby_no_arm_macro.xacro (robot description, xacro)
@@ -682,4 +682,44 @@
 		<origin rpy="1.57079619722 0 -1.57079632679" xyz="-0.035 -0.474758386705 0.592669"/>
     </joint>
+    <link name="tanks">
+        <visual>
+            <geometry>
+                <cylinder radius="0.0275" length="0.50" />
+            </geometry>
+			<material name="metal">
+				<color rgba="0.752941 0.752941 0.752941 1"/>
+            </material>
+        </visual>
+        <collision>
+            <geometry>
+                <cylinder radius="0.0275" length="0.50" />
+            </geometry>
+        </collision>
+    </link>
+    <joint name="frame-tanks" type="fixed">
+        <parent link="frame1"/>
+        <child link="tanks"/>
+		<origin rpy="0 0 0" xyz="0.16 -0.45 0.95"/>
+    </joint>
+    <link name="light">
+        <visual>
+            <geometry>
+                <cylinder radius="0.075" length="0.165" />
+            </geometry>
+			<material name="translucent_orange">
+        			<color rgba="1 0.43 0 0.5" />
+            </material>
+        </visual>
+        <collision>
+            <geometry>
+                <cylinder radius="0.075" length="0.165" />
+            </geometry>
+        </collision>
+    </link>
+    <joint name="frame-light" type="fixed">
+        <parent link="frame1"/>
+        <child link="light"/>
+		<origin rpy="0 1.571 0" xyz="0.215 -0.45 1.3"/>
+    </joint>
   </xacro:macro>
 </robot>
