Commit message: Trial 18.
Changed gripper_body collision shape to cylinder that encompasses
gripper jaws.
Commented out debug statement in twist receiver.

File: abby_description/urdf/gripper_macro.xacro (robot description, xacro)
@@ -19,7 +19,9 @@
 		<collision>
 			<geometry>
-				<mesh filename="package://abby_description/meshes/gripper_body.stl" scale="0.0254 0.0254 0.0254"/>
+			    <cylinder radius="0.04" length="0.13" />
+				<!--mesh filename="package://abby_description/meshes/gripper_body.stl" scale="0.0254 0.0254 0.0254"/-->
 			</geometry>
-			<origin rpy="3.141592653 0 0" xyz="0 0 0.017"/>
+			<origin rpy="0 0 0" xyz="0 0 0.065"/>
+			<!--origin rpy="3.141592653 0 0" xyz="0 0 0.017"/-->
 		</collision>
 	</link>

Commit message: Increases gripper collision size.
Increases length of gripper body collision box from 13 to 15 cm.
This should hopefully fix issues w/ gripper colliding with table.

File: abby_description/urdf/gripper_macro.xacro (robot description, xacro)
@@ -19,5 +19,5 @@
 		<collision>
 			<geometry>
-			    <box size="0.08 0.08 0.13" />
+			    <box size="0.08 0.08 0.15" />
 			    <!--cylinder radius="0.04" length="0.13" /-->
 				<!--mesh filename="package://abby_description/meshes/gripper_body.stl" scale="0.0254 0.0254 0.0254"/-->
