Commit message: Added gripper to the model.
Created a xacro macro for the gripper and added it to the model.
I may have to change the offset from the body to the gripper jaws,
which looks too large. All other measures should be correct. Effort
and velocity limits are bogus, but required by the model dtd.

Also altered show_model so that it doesn't try to launch the kinect.

File: abby_description/urdf/abby.xacro (robot description, xacro)
@@ -3,6 +3,8 @@
 	<include filename="$(find abb_common)/urdf/irb_120_macro.xacro" />
 	<include filename="$(find abby_description)/urdf/abby_no_arm_macro.xacro" />
+	<include filename="$(find abby_description)/urdf/gripper_macro.xacro" />
 	<xacro:irb_120 prefix="irb_120_"/>
     <xacro:abby_no_arm />
+    <xacro:abby_gripper />
     <joint name="frame_arm" type="fixed">
         <parent link="frame1"/>
@@ -10,3 +12,8 @@
 		<origin rpy="3.1415926535 1.57079632679 0" xyz="0.046 -0.55 .75"/>
     </joint>
+    <joint name="arm_gripper" type="fixed">
+        <parent link="irb_120_link_6"/>
+        <child link="gripper_body"/>
+		<origin rpy="0 0 0" xyz="0 0 0"/>
+    </joint>
 </robot>

File: abby_description/urdf/gripper.urdf (robot description, URDF)
Before this commit: robot abby, 41 links, 40 joints
Joints:
- joint arm_gripper: child gripper_body -> irb_120_base_link; parent irb_120_link_6 -> frame1

File: abby_description/urdf/gripper_macro.xacro (robot description, xacro)
@@ -7,5 +7,5 @@
 				<mesh filename="package://abby_description/meshes/gripper_body.stl" scale="0.0254 0.0254 0.0254"/>
 			</geometry>
-			<origin rpy="0 0 0" xyz="0.987350237145 0.252969532498 0.91153488"/>
+			<origin rpy="3.141592653 0 0" xyz="0 0 0.02497074"/>
 			<material name="gripper:21_color">
 				<color rgba="0.752941 0.752941 0.752941 1"/>
@@ -15,5 +15,5 @@
 			<mass value="0.222800943405"/>
 			<inertia ixx="0.000113884956016" ixy="0.0" ixz="0.0" iyy="0.000132512764251" iyz="-4.2661207134e-07" izz="9.078477651e-05"/>
-			<origin rpy="0 0 0" xyz="0.98735053139 0.252880388029 0.89481914"/>
+			<origin rpy="3.141592653 0 0" xyz="0 0 0.008255"/>
 		</inertial>
 		<collision>
@@ -21,5 +21,27 @@
 				<mesh filename="package://abby_description/meshes/gripper_body.stl" scale="0.0254 0.0254 0.0254"/>
 			</geometry>
-			<origin rpy="0 0 0" xyz="0.987350237145 0.252969532498 0.91153488"/>
+			<origin rpy="3.141592653 0 0" xyz="0 0 0.02497074"/>
+		</collision>
+	</link>
+	<link name="gripper_jaw_1">
+		<visual>
+			<geometry>
+				<mesh filename="package://abby_description/meshes/gripper_jaw.stl" scale="0.0254 0.0254 0.0254"/>
+			</geometry>
+			<origin rpy="1.570796327 0 0" xyz="0 0.0127 0"/>
+			<material name="gripper jaw:11_color">
+				<color rgba="0.752941 0.752941 0.752941 1"/>
+			</material>
+		</visual>
+		<inertial>
+			<mass value="0.00921754126924"/>
+			<inertia ixx="2.06132039615e-06" ixy="3.0409666492e-07" ixz="0.0" iyy="8.2195587923e-07" iyz="0.0" izz="1.7163745324e-06"/>
+			<origin rpy="0 0 0" xyz="0.006162341 0.03123184 0.0127004023"/>
+		</inertial>
+		<collision>
+			<geometry>
+				<mesh filename="package://abby_description/meshes/gripper_jaw.stl" scale="0.0254 0.0254 0.0254"/>
+			</geometry>
+			<origin rpy="1.570796327 0 0" xyz="0 0.0127 0"/>
 		</collision>
 	</link>
@@ -29,27 +51,5 @@
 				<mesh filename="package://abby_description/meshes/gripper_jaw.stl" scale="0.0254 0.0254 0.0254"/>
 			</geometry>
-			<origin rpy="0 0 0" xyz="-0.00616234095847 -0.01853184 -0.0127004918295"/>
-			<material name="gripper jaw:21_color">
-				<color rgba="0.752941 0.752941 0.752941 1"/>
-			</material>
-		</visual>
-		<inertial>
-			<mass value="0.00921754126924"/>
-			<inertia ixx="2.06132039615e-06" ixy="3.0409666492e-07" ixz="0.0" iyy="8.2195587923e-07" iyz="0.0" izz="1.7163745324e-06"/>
-			<origin rpy="0 0 0" xyz="0 0 0"/>
-		</inertial>
-		<collision>
-			<geometry>
-				<mesh filename="package://abby_description/meshes/gripper_jaw.stl" scale="0.0254 0.0254 0.0254"/>
-			</geometry>
-			<origin rpy="0 0 0" xyz="-0.00616234095847 -0.01853184 -0.0127004918295"/>
-		</collision>
-	</link>
-	<link name="gripper_jaw_1">
-		<visual>
-			<geometry>
-				<mesh filename="package://abby_description/meshes/gripper_jaw.stl" scale="0.0254 0.0254 0.0254"/>
-			</geometry>
-			<origin rpy="0 0 0" xyz="-0.00634967993098 -0.015875 0"/>
+			<origin rpy="1.570796327 0 0" xyz="0 0.0127 0"/>
 			<material name="gripper jaw:11_color">
 				<color rgba="0.752941 0.752941 0.752941 1"/>
@@ -59,5 +59,5 @@
 			<mass value="0.00921754126924"/>
 			<inertia ixx="2.06132039615e-06" ixy="3.0409666492e-07" ixz="0.0" iyy="8.2195587923e-07" iyz="0.0" izz="1.7163745324e-06"/>
-			<origin rpy="0 0 0" xyz="-0.000187338972516 0.00265684 0.0127004023134"/>
+			<origin rpy="0 0 0" xyz="0.006162341 0.03123184 0.0127004023"/>
 		</inertial>
 		<collision>
@@ -65,16 +65,18 @@
 				<mesh filename="package://abby_description/meshes/gripper_jaw.stl" scale="0.0254 0.0254 0.0254"/>
 			</geometry>
-			<origin rpy="0 0 0" xyz="-0.00634967993098 -0.015875 0"/>
+			<origin rpy="1.570796327 0 0" xyz="0 0.0127 0"/>
 		</collision>
 	</link>
-	<joint name="gripper_body--gripper_jaw_2" type="prismatic">
+	<joint name="gripper__jaw_1" type="prismatic">
+		<parent link="gripper_body"/>
+		<child link="gripper_jaw_1"/>
+		<origin rpy="0 0 3.14159265359" xyz="0 0 0.07699"/>
+		<limit upper="-0.022225" lower="-0.03175" effort="1" velocity="1" />
+	</joint>
+	<joint name="gripper_jaw_2" type="prismatic">
 		<parent link="gripper_body"/>
 		<child link="gripper_jaw_2"/>
-		<origin rpy="-1.57079632679 0 3.14159265359" xyz="1.02008231217 0.253784397197 0.85691472"/>
-	</joint>
-	<joint name="gripper_jaw_2 -- gripper_jaw_1" type="prismatic">
-		<parent link="gripper_jaw_2"/>
-		<child link="gripper_jaw_1"/>
-		<origin rpy="3.14159265359 0 -3.14159265359" xyz="0.0652760334972 -0.00265684 0.0126998117907"/>
+		<origin rpy="0 0 0" xyz="0 0 0.07699"/>
+		<limit upper="-0.022225" lower="-0.03175" effort="1" velocity="1" />
 	</joint>
   </xacro:macro>

Commit message: Fixes arm location.
The arm was offset by several cm in the x direction and a few mm in the
y and z direction. Corrections were made by taking the x and y coordinates
from the kinect and lidar respectively and by lowering the arm as far as
possible and measuring the distance from gripper tip to floor to correct
the z.
(All coordinates above in /base_link frame.)

File: abby_description/urdf/abby.xacro (robot description, xacro)
@@ -10,5 +10,5 @@
         <parent link="frame1"/>
         <child link="irb_120_base_link"/>
-		<origin rpy="3.1415926535 1.57079632679 0" xyz="0.046 -0.55 .75"/>
+		<origin rpy="3.1415926535 1.57079632679 0" xyz="0.04464 -0.475 0.703"/>
     </joint>
     <joint name="arm_gripper" type="fixed">

Commit message: Fixed kinect and arm frames.
Kinect now publishes frames for rgb and depth in the correct
place. (curse you willowgarage).

IRB-120 has been moved and rotated to reflect the fact that the rail it is
mounted to is not actually vertical. A more complete fix would be to rotate
the whole frame in the model to be correct, but this will do for now.

File: abby_description/urdf/abby.xacro (robot description, xacro)
@@ -10,5 +10,5 @@
         <parent link="frame1"/>
         <child link="irb_120_base_link"/>
-		<origin rpy="3.1415926535 1.57079632679 0" xyz="0.04464 -0.475 0.703"/>
+		<origin rpy="-1.571 1.446 1.571" xyz="0.04464 -0.473311 0.753907"/>
     </joint>
     <joint name="arm_gripper" type="fixed">

Commit message: Moved the arm back again.
Seems like the arm wasn't as tilted as I thought. Moved it back to
being flush with the rail and it's pretty close to correct.

File: abby_description/urdf/abby.xacro (robot description, xacro)
@@ -10,5 +10,6 @@
         <parent link="frame1"/>
         <child link="irb_120_base_link"/>
-		<origin rpy="-1.571 1.446 1.571" xyz="0.04464 -0.473311 0.753907"/>
+		<origin rpy="3.14159 1.571 0" xyz="0.046 -0.47 0.70"/>
+		<!--origin rpy="-1.571 1.446 1.571" xyz="0.04464 -0.473311 0.753907"/-->
     </joint>
     <joint name="arm_gripper" type="fixed">

Commit message: Realligned the arm.
This time with more linear algebra.
The result is plausible, and looks good for some arm positions,
but not for others. For the 18 points it's calculated from, it has
RMS position error of 1.4 cm. However, the misallignment of the
meshes is obvious in rviz. I suspect the Kinect is nonlinear and
inaccurate.

File: abby_description/urdf/abby.xacro (robot description, xacro)
@@ -7,8 +7,8 @@
     <xacro:abby_no_arm />
     <xacro:abby_gripper />
-    <joint name="frame_arm" type="fixed">
-        <parent link="frame1"/>
+    <joint name="camera_arm" type="fixed">
+        <parent link="camera_rgb_optical_frame"/>
         <child link="irb_120_base_link"/>
-		<origin rpy="3.14159 1.571 0" xyz="0.046 -0.47 0.70"/>
+		<origin rpy="1.641 -0.821 1.582" xyz="-.0310 .575028 .52330"/>
 		<!--origin rpy="-1.571 1.446 1.571" xyz="0.04464 -0.473311 0.753907"/-->
     </joint>

Commit message: Another attempt at getting the kinect->arm transform right.
It still isn't right, but this is based on points near the table. I guess I need more points

File: abby_description/urdf/abby.xacro (robot description, xacro)
@@ -7,8 +7,9 @@
     <xacro:abby_no_arm />
     <xacro:abby_gripper />
-    <joint name="camera_arm" type="fixed">
-        <parent link="camera_rgb_optical_frame"/>
+	<xacro:kinect xyz="0.04464 -0.59 1.491" rpy="0 0.8901 -1.570795" parent_frame="frame1" />
+    <joint name="frame_arm" type="fixed">
+        <parent link="frame1"/>
         <child link="irb_120_base_link"/>
-		<origin rpy="1.641 -0.821 1.582" xyz="-.0310 .575028 .52330"/>
+		<origin rpy="0.439 1.505 -2.649" xyz="0.033 -0.477 0.674"/>
 		<!--origin rpy="-1.571 1.446 1.571" xyz="0.04464 -0.473311 0.753907"/-->
     </joint>

File: abby_description/urdf/abby_no_arm_macro.xacro (robot description, xacro)
@@ -4,5 +4,4 @@
     <include filename="$(find cwru_description)/urdf/sick_LMS291.urdf.xacro"/>
 	<xacro:macro name="abby_no_arm">
-	  <xacro:kinect xyz="0.04464 -0.59 1.491" rpy="0 0.8901 -1.570795" parent_frame="frame1" />
 	  <xacro:SICK_LMS291 parent_frame="frame1" laser_frame="base_laser1_link" rpy="1.5707959092 0 -3.14159265358" xyz="-0.0255468119868 -0.474758386705 0.311455920061"/>
 	  <link name="frame1">

Commit message: Changes to arm configuration.
Moves arm up 85 mm and aligns w/ kinect. Alignment is still off in the
xy plane (rotation and/or translation).

Configures ompl planning to use monitor and increases self filter padding.

File: abby_description/urdf/abby.xacro (robot description, xacro)
@@ -11,6 +11,7 @@
         <parent link="frame1"/>
         <child link="irb_120_base_link"/>
-		<origin rpy="0.439 1.505 -2.649" xyz="0.033 -0.477 0.674"/>
-		<!--origin rpy="-1.571 1.446 1.571" xyz="0.04464 -0.473311 0.753907"/-->
+        <!--origin rpy="0.439 1.505 -2.649" xyz="0.033 -0.477 0.674" /-->
+		<origin rpy="3.142 1.571 0" xyz="0.033 -0.477 0.760" />
+		<!--origin rpy="0.439 1.505 -2.649" xyz="0.033 -0.477 0.674" /-->
     </joint>
     <joint name="arm_gripper" type="fixed">

Commit message: Trial 39
Fixed grasp angle for boxes that are only pickable along the y axis
Realligned arm.

File: abby_description/urdf/abby.xacro (robot description, xacro)
@@ -8,10 +8,10 @@
     <xacro:abby_gripper />
 	<xacro:kinect xyz="0.04464 -0.59 1.491" rpy="0 0.8901 -1.570795" parent_frame="frame1" />
-    <joint name="frame_arm" type="fixed">
+    <joint name="frame_arm" type="fixed" >
+        <axis xyz="1 0 0"/>
         <parent link="frame1"/>
         <child link="irb_120_base_link"/>
-        <!--origin rpy="0.439 1.505 -2.649" xyz="0.033 -0.477 0.674" /-->
-		<origin rpy="3.142 1.571 0" xyz="0.033 -0.477 0.760" />
-		<!--origin rpy="0.439 1.505 -2.649" xyz="0.033 -0.477 0.674" /-->
+		<origin rpy="0.060 1.571 -3.142" xyz="0.05 -0.477 0.780" />
+		<!-- origin rpy="3.142 1.571 0" xyz="0.033 -0.477 0.760" /-->
     </joint>
     <joint name="arm_gripper" type="fixed">

Commit message: Trial 40
Arm finally aligned. Successfully picked a box.

File: abby_description/urdf/abby.xacro (robot description, xacro)
@@ -12,6 +12,8 @@
         <parent link="frame1"/>
         <child link="irb_120_base_link"/>
-		<origin rpy="0.060 1.571 -3.142" xyz="0.05 -0.477 0.780" />
-		<!-- origin rpy="3.142 1.571 0" xyz="0.033 -0.477 0.760" /-->
+		<origin rpy="-0.069 1.542 3.028" xyz="0.051 -0.489 0.760" />
+		<!--origin rpy="-0.572 1.525 2.433" xyz="0.085 -0.507 0.771" /-->
+		<!--origin rpy="-0.055 1.571 -3.142" xyz="0.02 -0.477 0.780" /-->
+		<!--origin rpy="3.142 1.571 0" xyz="0.033 -0.477 0.760" /-->
     </joint>
     <joint name="arm_gripper" type="fixed">

Commit message: Alignment for new kinect.

File: abby_description/urdf/abby.xacro (robot description, xacro)
@@ -7,14 +7,38 @@
     <xacro:abby_no_arm />
     <xacro:abby_gripper />
-	<xacro:kinect xyz="0.04464 -0.59 1.491" rpy="0 0.8901 -1.570795" parent_frame="frame1" />
-    <joint name="frame_arm" type="fixed" >
-        <axis xyz="1 0 0"/>
-        <parent link="frame1"/>
-        <child link="irb_120_base_link"/>
-		<origin rpy="-0.069 1.542 3.028" xyz="0.051 -0.489 0.760" />
+	<xacro:kinect xyz="0.508 -0.035 1.601" rpy="0.045 0.880 0.0" parent_frame="base_link" />
+	<link name="base_link">
+	</link>
+	<link name="dummy">
+	</link>
+	<joint name="base_joint" type="fixed">
+	    <parent link="base_link"/>
+	    <origin rpy="0 0 1.570795" xyz="-0.07963916 -0.04203954 0.11" />
+	    <child link="frame1"/>
+	</joint>
+	<joint name="base_dummy" type="fixed" >
+	    <parent link="base_link" />
+	    <child link="dummy" />
+	    <!--origin xyz="0.377 -0.078 0.869" rpy="3.005 1.553 1.541" /--> <!-- 1-10 -->
+	    <!--origin xyz="0.362 -0.067 0.868" rpy="0.361 1.521 -1.171" /--> <!-- 11-20 -->
+	    <!--origin xyz="0.371 -0.058 0.860" rpy="0.479 1.527 -1.046" /-->  <!-- 1-20 -->
+	    <!--origin xyz="0.378 -0.019 0.855" rpy="1.693 1.547 0.098" /-->  <!-- 1-30 -->
+	    <!--origin xyz="0.380 -0.031 0.878" rpy="-2.510 1.546 2.197" /-->  <!-- 1-40 -->
+	    <origin xyz="0.380 0.008 0.858" rpy="2.156 1.514 0.481" /> <!-- 1-45 -->
+	</joint>
+	<joint name="dummy_arm" type="fixed" >
+	    <parent link="dummy" />
+	    <child link="irb_120_base_link" />
+	    <origin xyz="-.01 0 0" rpy="0 0 -0.05" />
+	</joint>
+    <!--joint name="frame_arm" type="fixed" -->
+        <!--axis xyz="1 0 0"/-->
+        <!--parent link="frame1"/-->
+        <!--child link="irb_120_base_link"/-->
+		<!--origin rpy="-0.069 1.542 3.028" xyz="0.051 -0.489 0.760" /-->
 		<!--origin rpy="-0.572 1.525 2.433" xyz="0.085 -0.507 0.771" /-->
 		<!--origin rpy="-0.055 1.571 -3.142" xyz="0.02 -0.477 0.780" /-->
 		<!--origin rpy="3.142 1.571 0" xyz="0.033 -0.477 0.760" /-->
-    </joint>
+    <!--/joint-->
     <joint name="arm_gripper" type="fixed">
         <parent link="irb_120_link_6"/>

File: abby_description/urdf/gripper_macro.xacro (robot description, xacro)
@@ -19,5 +19,6 @@
 		<collision>
 			<geometry>
-			    <cylinder radius="0.04" length="0.13" />
+			    <box size="0.08 0.08 0.13" />
+			    <!--cylinder radius="0.04" length="0.13" /-->
 				<!--mesh filename="package://abby_description/meshes/gripper_body.stl" scale="0.0254 0.0254 0.0254"/-->
 			</geometry>

Commit message: Arm alignment (this time for realz).

File: abby_description/urdf/abby.xacro (robot description, xacro)
@@ -20,15 +20,10 @@
 	    <parent link="base_link" />
 	    <child link="dummy" />
-	    <!--origin xyz="0.377 -0.078 0.869" rpy="3.005 1.553 1.541" /--> <!-- 1-10 -->
-	    <!--origin xyz="0.362 -0.067 0.868" rpy="0.361 1.521 -1.171" /--> <!-- 11-20 -->
-	    <!--origin xyz="0.371 -0.058 0.860" rpy="0.479 1.527 -1.046" /-->  <!-- 1-20 -->
-	    <!--origin xyz="0.378 -0.019 0.855" rpy="1.693 1.547 0.098" /-->  <!-- 1-30 -->
-	    <!--origin xyz="0.380 -0.031 0.878" rpy="-2.510 1.546 2.197" /-->  <!-- 1-40 -->
-	    <origin xyz="0.380 0.008 0.858" rpy="2.156 1.514 0.481" /> <!-- 1-45 -->
+	    <origin xyz="0.379 0.008 0.858" rpy="3.142 1.571 1.571" />
 	</joint>
 	<joint name="dummy_arm" type="fixed" >
 	    <parent link="dummy" />
 	    <child link="irb_120_base_link" />
-	    <origin xyz="-.01 0 0" rpy="0 0 -0.05" />
+	    <origin xyz="-0.03 .01 0.035" rpy="0.025 0.032 -0.05" />
 	</joint>
     <!--joint name="frame_arm" type="fixed" -->

Commit message: Somewhat better alignment.
Arm alignment from linear regression on 25 points.

File: abby_description/urdf/abby.xacro (robot description, xacro)
@@ -25,5 +25,8 @@
 	    <parent link="dummy" />
 	    <child link="irb_120_base_link" />
-	    <origin xyz="-0.03 .01 0.035" rpy="0.025 0.032 -0.05" />
+	    <!--origin xyz="-0.032 -0.006 0.043" rpy="0.026 0.025 -0.047" /--> <!-- 1-10, 21-25 -->
+	    <!--origin xyz="-0.028 -0.006 0.040" rpy="0.026 0.015 -0.044" /--> <!-- 1-10, 16-25 -->
+	    <origin xyz="-0.028 -0.006 0.040" rpy="0.026 0.015 -0.044" /> <!-- 1-10, 16-30 -->
+	    <!--origin xyz="-0.03 .01 0.035" rpy="0.025 0.032 -0.05" /--> <!--Visually aligned -->
 	</joint>
     <!--joint name="frame_arm" type="fixed" -->

Commit message: Manipulation demos.
This is the code used for manipulation demos.
Arm position tweaked over by a few mm.
Manipulation demo now includes driving up to table (so collision map
has full table in it.)

File: abby_description/urdf/abby.xacro (robot description, xacro)
@@ -27,5 +27,6 @@
 	    <!--origin xyz="-0.032 -0.006 0.043" rpy="0.026 0.025 -0.047" /--> <!-- 1-10, 21-25 -->
 	    <!--origin xyz="-0.028 -0.006 0.040" rpy="0.026 0.015 -0.044" /--> <!-- 1-10, 16-25 -->
-	    <origin xyz="-0.028 -0.006 0.040" rpy="0.026 0.015 -0.044" /> <!-- 1-10, 16-30 -->
+	    <!--origin xyz="-0.028 -0.006 0.040" rpy="0.026 0.015 -0.044" /--> <!-- 1-10, 16-30 -->
+	    <origin xyz="-0.028 -0.006 0.036" rpy="0.026 0.015 -0.044" /> <!-- 1-10, 16-30, tweaked -->
 	    <!--origin xyz="-0.03 .01 0.035" rpy="0.025 0.032 -0.05" /--> <!--Visually aligned -->
 	</joint>

Commit message: Day 2 trials, model edits. (committed before M30)
Moves arm 1 mm to left.
Replaces compressor collision mesh with a box that encompasses
the valve and gauge assembly.
Increases the length of the gripper collision box.

File: abby_description/urdf/abby.xacro (robot description, xacro)
@@ -28,5 +28,5 @@
 	    <!--origin xyz="-0.028 -0.006 0.040" rpy="0.026 0.015 -0.044" /--> <!-- 1-10, 16-25 -->
 	    <!--origin xyz="-0.028 -0.006 0.040" rpy="0.026 0.015 -0.044" /--> <!-- 1-10, 16-30 -->
-	    <origin xyz="-0.028 -0.006 0.036" rpy="0.026 0.015 -0.044" /> <!-- 1-10, 16-30, tweaked -->
+	    <origin xyz="-0.028 -0.006 0.035" rpy="0.026 0.015 -0.044" /> <!-- 1-10, 16-30, tweaked -->
 	    <!--origin xyz="-0.03 .01 0.035" rpy="0.025 0.032 -0.05" /--> <!--Visually aligned -->
 	</joint>

File: abby_description/urdf/abby_no_arm_macro.xacro (robot description, xacro)
@@ -341,7 +341,9 @@
 		<collision>
 			<geometry>
-				<mesh filename="package://abby_description/meshes/compressor_iam_e870b89.stl" scale="0.0254 0.0254 0.0254"/>
-			</geometry>
-			<origin rpy="0 0 0" xyz="0.217095026073 0.0541649919903 0.058507418554"/>
+			    <box size="0.26 0.12 0.27" />
+				<!--mesh filename="package://abby_description/meshes/compressor_iam_e870b89.stl" scale="0.0254 0.0254 0.0254"/-->
+			</geometry>
+			<origin rpy="0 0 0" xyz="0.13 0 -0.015"/> <!-- For box -->
+			<!--origin rpy="0 0 0" xyz="0.217095026073 0.0541649919903 0.058507418554"/--> <!--For mesh -->
 		</collision>
 	</link>

File: abby_description/urdf/gripper_macro.xacro (robot description, xacro)
@@ -19,5 +19,5 @@
 		<collision>
 			<geometry>
-			    <box size="0.08 0.08 0.15" />
+			    <box size="0.08 0.08 0.13" />
 			    <!--cylinder radius="0.04" length="0.13" /-->
 				<!--mesh filename="package://abby_description/meshes/gripper_body.stl" scale="0.0254 0.0254 0.0254"/-->

Commit message: Honestly, I'm not even sure. Final manipulation demo.
This is the final manipulation demo code. Not sure what changed
here.`

File: abby_description/urdf/abby.xacro (robot description, xacro)
@@ -7,5 +7,5 @@
     <xacro:abby_no_arm />
     <xacro:abby_gripper />
-	<xacro:kinect xyz="0.508 -0.035 1.601" rpy="0.045 0.880 0.0" parent_frame="base_link" />
+	<xacro:kinect xyz="0.508 -0.010 1.601" rpy="0.045 0.880 0.0" parent_frame="base_link" />
 	<link name="base_link">
 	</link>
@@ -20,5 +20,5 @@
 	    <parent link="base_link" />
 	    <child link="dummy" />
-	    <origin xyz="0.379 0.008 0.858" rpy="3.142 1.571 1.571" />
+	    <origin xyz="0.379 0.033 0.858" rpy="3.142 1.571 1.571" />
 	</joint>
 	<joint name="dummy_arm" type="fixed" >
@@ -28,5 +28,5 @@
 	    <!--origin xyz="-0.028 -0.006 0.040" rpy="0.026 0.015 -0.044" /--> <!-- 1-10, 16-25 -->
 	    <!--origin xyz="-0.028 -0.006 0.040" rpy="0.026 0.015 -0.044" /--> <!-- 1-10, 16-30 -->
-	    <origin xyz="-0.028 -0.006 0.035" rpy="0.026 0.015 -0.044" /> <!-- 1-10, 16-30, tweaked -->
+	    <origin xyz="-0.028 -0.006 0.038" rpy="0.026 0.015 -0.044" /> <!-- 1-10, 16-30, tweaked -->
 	    <!--origin xyz="-0.03 .01 0.035" rpy="0.025 0.032 -0.05" /--> <!--Visually aligned -->
 	</joint>
