Commit message: Melodic branch started
This is an update so get this back working for Melodic.  The base is controlled with the diff_drive controller and can be teloperated with a joystick.  The Kinect and SICK lidar elements are visible, but the drivers are not yet tested.

File: abby_description/urdf/abby.xacro (robot description, xacro)
@@ -1,11 +1,16 @@
 <?xml version="1.0" ?>
 <robot name="abby" xmlns:xacro="http://ros.org/wiki/xacro">
-	<include filename="$(find abb_common)/urdf/irb_120_macro.xacro" />
-	<include filename="$(find abby_description)/urdf/abby_no_arm_macro.xacro" />
-	<include filename="$(find abby_description)/urdf/gripper_macro.xacro" />
+	<xacro:include filename="$(find abb_common)/urdf/irb_120_macro.xacro" />
+	<xacro:include filename="$(find abby_description)/urdf/abby_base_macro.xacro" />
+	<xacro:include filename="$(find abby_description)/urdf/abby_gripper_macro.xacro" />
+	<xacro:property name="M_PI" value="${pi}" />
+	<xacro:include filename="$(find abby_description)/urdf/abby_gazebo.xacro" />
+	<!-- <xacro:include filename="$(find abby_description)/urdf/kinect_calibration.xacro" /> -->
+	<xacro:include filename="$(find openni_description)/model/kinect.urdf.xacro" />
 	<xacro:irb_120 prefix="irb_120_"/>
-    <xacro:abby_no_arm />
+    <xacro:abby_base />
     <xacro:abby_gripper />
-	<xacro:kinect xyz="0.508 -0.010 1.601" rpy="0.045 0.880 0.0" parent_frame="base_link" />
+	<xacro:sensor_kinect cam_px="0.508" cam_py="-0.010" cam_pz="1.601" cam_or="0.045" cam_op="0.880" cam_oy="0.0" parent="base_link" />
+	<!-- <xacro:sensor_kinect cam_px="kinect_calib_cam_x" cam_py="kinect_calib_cam_y" cam_pz="kinect_calib_cam_z" cam_or="kinect_calib_cam_rr" cam_op="kinect_calib_cam_rp" cam_oy="kinect_calib_cam_ry" parent="base_link" /> -->
 	<link name="base_link">
 	</link>
@@ -31,13 +36,4 @@
 	    <!--origin xyz="-0.03 .01 0.035" rpy="0.025 0.032 -0.05" /--> <!--Visually aligned -->
 	</joint>
-    <!--joint name="frame_arm" type="fixed" -->
-        <!--axis xyz="1 0 0"/-->
-        <!--parent link="frame1"/-->
-        <!--child link="irb_120_base_link"/-->
-		<!--origin rpy="-0.069 1.542 3.028" xyz="0.051 -0.489 0.760" /-->
-		<!--origin rpy="-0.572 1.525 2.433" xyz="0.085 -0.507 0.771" /-->
-		<!--origin rpy="-0.055 1.571 -3.142" xyz="0.02 -0.477 0.780" /-->
-		<!--origin rpy="3.142 1.571 0" xyz="0.033 -0.477 0.760" /-->
-    <!--/joint-->
     <joint name="arm_gripper" type="fixed">
         <parent link="irb_120_link_6"/>

File: abby_description/urdf/kinect_calibration.xacro (robot description, xacro)
@@ -1,10 +1,10 @@
 <?xml version="1.0"?>
 <robot>
-  <property name="kinect_calib_cam_x" value="-0.0844382" />
-  <property name="kinect_calib_cam_y" value="0" />
-  <property name="kinect_calib_cam_z" value="0.1047496" />
-  <property name="kinect_calib_cam_rr" value="0" />
-  <property name="kinect_calib_cam_rp" value="0" />
-  <property name="kinect_calib_cam_ry" value="0" />
-  <property name="kinect_camera_parent_name" value="frame1" />
+  <xacro:property name="kinect_calib_cam_x" value="-0.0844382" />
+  <xacro:property name="kinect_calib_cam_y" value="0" />
+  <xacro:property name="kinect_calib_cam_z" value="0.1047496" />
+  <xacro:property name="kinect_calib_cam_rr" value="0" />
+  <xacro:property name="kinect_calib_cam_rp" value="0" />
+  <xacro:property name="kinect_calib_cam_ry" value="0" />
+  <xacro:property name="kinect_camera_parent_name" value="frame1" />
 </robot>
